File: hardware/electronics/sensori-linea/sensori di linea /sensori di linea soccer 2018.sch (EAGLE design)
At the start: 21 parts, among them T1 BP103, T2 BP103, T3 BP103, T4 BP103

Commit message: miglioramenti sensori di linea 2018
Parts:
- removed D1, D2, D3, D4: WHITE, SparkFun-LED:LED-WHITE1206
- added D5, D6, D7, D8: (no value), SparkFun-LED:LED3MM
Connections:
- net GND: now also D5.C, D6.C, D7.C, D8.C; no longer D1.C, D2.C, D3.C, D4.C
- net N$2: now also D5.A; no longer D1.A
- net N$3: now also D6.A; no longer D2.A
- net N$4: now also D7.A; no longer D3.A
- net N$5: now also D8.A; no longer D4.A
Changed lines of the file:
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@@
 <part name="C3" library="SparkFun-Capacitors" deviceset="3.3NF" device="-0603-100V-10%" value="3.3nF"/>
 <part name="C4" library="SparkFun-Capacitors" deviceset="3.3NF" device="-0603-100V-10%" value="3.3nF"/>
-<part name="D1" library="SparkFun-LED" deviceset="LED-WHITE" device="1206" value="WHITE"/>
-<part name="D2" library="SparkFun-LED" deviceset="LED-WHITE" device="1206" value="WHITE"/>
-<part name="D3" library="SparkFun-LED" deviceset="LED-WHITE" device="1206" value="WHITE"/>
-<part name="D4" library="SparkFun-LED" deviceset="LED-WHITE" device="1206" value="WHITE"/>
 <part name="FRAME1" library="frames" library_urn="urn:adsk.eagle:library:229" deviceset="A3L-LOC" device=""/>
+<part name="D5" library="SparkFun-LED" deviceset="LED" device="3MM"/>
+<part name="D6" library="SparkFun-LED" deviceset="LED" device="3MM"/>
+<part name="D7" library="SparkFun-LED" deviceset="LED" device="3MM"/>
+<part name="D8" library="SparkFun-LED" deviceset="LED" device="3MM"/>
 </parts>
 <sheets>
@@
 <instance part="C3" gate="G$1" x="139.7" y="162.56"/>
 <instance part="C4" gate="G$1" x="86.36" y="162.56"/>
-<instance part="D1" gate="G$1" x="177.8" y="185.42"/>
-<instance part="D2" gate="G$1" x="187.96" y="185.42"/>
-<instance part="D3" gate="G$1" x="198.12" y="185.42"/>
-<instance part="D4" gate="G$1" x="208.28" y="185.42"/>
 <instance part="FRAME1" gate="G$1" x="33.02" y="-5.08"/>
+<instance part="D5" gate="G$1" x="177.8" y="185.42"/>
+<instance part="D6" gate="G$1" x="187.96" y="185.42"/>
+<instance part="D7" gate="G$1" x="198.12" y="185.42"/>
+<instance part="D8" gate="G$1" x="208.28" y="185.42"/>
 </instances>
 <busses>
@@
 <junction x="193.04" y="175.26"/>
 <label x="193.04" y="170.18" size="1.778" layer="95" rot="R270" xref="yes"/>
-<pinref part="D1" gate="G$1" pin="C"/>
-<pinref part="D2" gate="G$1" pin="C"/>
-<pinref part="D3" gate="G$1" pin="C"/>
-<pinref part="D4" gate="G$1" pin="C"/>
+<pinref part="D5" gate="G$1" pin="C"/>
+<pinref part="D6" gate="G$1" pin="C"/>
+<pinref part="D7" gate="G$1" pin="C"/>
+<pinref part="D8" gate="G$1" pin="C"/>
 </segment>
 <segment>
@@
 <pinref part="R5" gate="G$1" pin="1"/>
 <wire x1="177.8" y1="190.5" x2="177.8" y2="187.96" width="0.1524" layer="91"/>
-<pinref part="D1" gate="G$1" pin="A"/>
+<pinref part="D5" gate="G$1" pin="A"/>
 </segment>
 </net>
@@
 <pinref part="R6" gate="G$1" pin="1"/>
 <wire x1="187.96" y1="190.5" x2="187.96" y2="187.96" width="0.1524" layer="91"/>
-<pinref part="D2" gate="G$1" pin="A"/>
+<pinref part="D6" gate="G$1" pin="A"/>
 </segment>
 </net>
@@
 <pinref part="R7" gate="G$1" pin="1"/>
 <wire x1="198.12" y1="190.5" x2="198.12" y2="187.96" width="0.1524" layer="91"/>
-<pinref part="D3" gate="G$1" pin="A"/>
+<pinref part="D7" gate="G$1" pin="A"/>
 </segment>
 </net>
@@
 <pinref part="R8" gate="G$1" pin="1"/>
 <wire x1="208.28" y1="190.5" x2="208.28" y2="187.96" width="0.1524" layer="91"/>
-<pinref part="D4" gate="G$1" pin="A"/>
-</segment>
-</net>
+<pinref part="D8" gate="G$1" pin="A"/>
+</segment>
+</net>
