File: hardware/electronics/sensori-linea/sensori di linea /sensori di linea soccer 2018.brd (EAGLE design)
At the start: 88.1 x 42 mm, 21 parts, among them T1 BP103, T2 BP103, T3 BP103, T4 BP103

Commit message: aggiornamenti sensori
Parts:
- added C5: 1.0uF, SparkFun-Capacitors:0402
- added R13, R14, R15, R16: (no value), resistor:0204/7
- added U$1: ADS1015IDGT, bt_adc:MSOP10_0.5
Connections:
- new net N$1: R13.1, U$1.1
- new net N$6: R16.2, U$1.9
- new net N$7: R14.2, U$1.2
- new net N$8: R15.2, U$1.10
- net GND: now also C5.2, R13.2, U$1.3
- net OUT1: now also U$1.4
- net OUT2: now also U$1.5
- net OUT3: now also U$1.6
- net OUT4: now also U$1.7
- net VCC: now also C5.1, R14.1, R15.1, R16.1, U$1.8
Changed lines of the file:
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@@
 <layers>
 <layer number="1" name="Top" color="4" fill="1" visible="yes" active="yes"/>
+<layer number="2" name="Route2" color="1" fill="3" visible="yes" active="yes"/>
+<layer number="3" name="Route3" color="4" fill="3" visible="yes" active="yes"/>
+<layer number="4" name="Route4" color="1" fill="4" visible="yes" active="yes"/>
+<layer number="5" name="Route5" color="4" fill="4" visible="yes" active="yes"/>
+<layer number="6" name="Route6" color="1" fill="8" visible="yes" active="yes"/>
+<layer number="7" name="Route7" color="4" fill="8" visible="yes" active="yes"/>
+<layer number="8" name="Route8" color="1" fill="2" visible="yes" active="yes"/>
+<layer number="9" name="Route9" color="4" fill="2" visible="yes" active="yes"/>
+<layer number="10" name="Route10" color="1" fill="7" visible="yes" active="yes"/>
+<layer number="11" name="Route11" color="4" fill="7" visible="yes" active="yes"/>
+<layer number="12" name="Route12" color="1" fill="5" visible="yes" active="yes"/>
+<layer number="13" name="Route13" color="4" fill="5" visible="yes" active="yes"/>
+<layer number="14" name="Route14" color="1" fill="6" visible="yes" active="yes"/>
+<layer number="15" name="Route15" color="4" fill="6" visible="yes" active="yes"/>
 <layer number="16" name="Bottom" color="1" fill="1" visible="yes" active="yes"/>
 <layer number="17" name="Pads" color="2" fill="1" visible="yes" active="yes"/>
@@
 <attribute name="PROD_ID" value="DIO-08794" x="-30.48" y="69.85" size="1.778" layer="28" font="vector" rot="MR180" display="off"/>
 </element>
+<element name="U$1" library="bt_adc" package="MSOP10_0.5" value="ADS1015IDGT" x="-24.13" y="52.07"/>
+<element name="C5" library="SparkFun-Capacitors" package="0402" value="1.0uF" x="-19.05" y="35.56">
+<attribute name="PROD_ID" value="CAP-12417" x="-19.05" y="35.56" size="1.778" layer="27" display="off"/>
+</element>
+<element name="R13" library="resistor" library_urn="urn:adsk.eagle:library:348" package="0204/7" package3d_urn="urn:adsk.eagle:package:25945/1" value="" x="-38.1" y="45.72"/>
+<element name="R14" library="resistor" library_urn="urn:adsk.eagle:library:348" package="0204/7" package3d_urn="urn:adsk.eagle:package:25945/1" value="" x="-38.1" y="39.37"/>
+<element name="R15" library="resistor" library_urn="urn:adsk.eagle:library:348" package="0204/7" package3d_urn="urn:adsk.eagle:package:25945/1" value="" x="-34.29" y="34.29"/>
+<element name="R16" library="resistor" library_urn="urn:adsk.eagle:library:348" package="0204/7" package3d_urn="urn:adsk.eagle:package:25945/1" value="" x="-38.1" y="49.53"/>
 </elements>
 <signals>
@@
 <wire x1="-20.32" y1="68.58" x2="-19.05" y2="69.85" width="0.6096" layer="16"/>
 <wire x1="-19.05" y1="69.85" x2="-10.16" y2="69.85" width="0.6096" layer="16"/>
+<contactref element="U$1" pad="8"/>
+<contactref element="C5" pad="1"/>
+<contactref element="R14" pad="1"/>
+<contactref element="R16" pad="1"/>
+<contactref element="R15" pad="1"/>
+<wire x1="-38.1" y1="34.29" x2="-41.91" y2="49.53" width="0" layer="19" extent="1-1"/>
+<wire x1="-41.91" y1="39.37" x2="-38.1" y2="34.29" width="0" layer="19" extent="1-1"/>
+<wire x1="-19.63" y1="35.56" x2="-41.91" y2="39.37" width="0" layer="19" extent="1-1"/>
+<wire x1="-24.13" y1="54.47" x2="-19.63" y2="35.56" width="0" layer="19" extent="1-1"/>
+<wire x1="-20.32" y1="67.31" x2="-24.13" y2="54.47" width="0" layer="19" extent="1-1"/>
 </signal>
 <signal name="OUT1">
@@
 <wire x1="-3.81" y1="60.96" x2="-3.81" y2="58.42" width="0.6096" layer="16"/>
 <wire x1="-3.81" y1="58.42" x2="-2.54" y2="57.15" width="0.6096" layer="16"/>
+<contactref element="U$1" pad="4"/>
+<wire x1="-23.63" y1="49.67" x2="-3.81" y2="53.34" width="0" layer="19" extent="1-16"/>
 </signal>
 <signal name="GND">
@@
 </polygon>
 <via x="26.67" y="66.04" extent="1-16" drill="0.35"/>
+<contactref element="U$1" pad="3"/>
+<contactref element="C5" pad="2"/>
+<contactref element="R13" pad="2"/>
+<wire x1="28.36" y1="66.04" x2="35.56" y2="73.66" width="0" layer="19" extent="1-1"/>
+<wire x1="26.67" y1="66.04" x2="28.36" y2="66.04" width="0" layer="19" extent="1-1"/>
+<wire x1="24.13" y1="69.85" x2="26.67" y2="66.04" width="0" layer="19" extent="1-1"/>
+<wire x1="19.05" y1="73.66" x2="24.13" y2="69.85" width="0" layer="19" extent="1-1"/>
+<wire x1="1.69" y1="66.04" x2="19.05" y2="73.66" width="0" layer="19" extent="1-1"/>
+<wire x1="-2.54" y1="68.58" x2="1.69" y2="66.04" width="0" layer="19" extent="1-1"/>
+<wire x1="-3.39" y1="66.04" x2="-2.54" y2="68.58" width="0" layer="19" extent="1-1"/>
+<wire x1="-10.16" y1="73.66" x2="-2.54" y2="68.58" width="0" layer="19" extent="1-1"/>
+<wire x1="-12.7" y1="72.39" x2="-10.16" y2="73.66" width="0" layer="19" extent="1-1"/>
+<wire x1="1.27" y1="54.61" x2="1.69" y2="66.04" width="0" layer="19" extent="1-1"/>
+<wire x1="-1.27" y1="46.99" x2="1.27" y2="54.61" width="0" layer="19" extent="1-1"/>
+<wire x1="-26.25" y1="66.04" x2="-12.7" y2="72.39" width="0" layer="19" extent="1-1"/>
+<wire x1="-29.21" y1="69.85" x2="-26.25" y2="66.04" width="0" layer="19" extent="1-1"/>
+<wire x1="-24.13" y1="49.67" x2="-26.25" y2="66.04" width="0" layer="19" extent="1-1"/>
+<wire x1="-18.47" y1="35.56" x2="-24.13" y2="49.67" width="0" layer="19" extent="1-1"/>
+<wire x1="-34.29" y1="45.72" x2="-18.47" y2="35.56" width="0" layer="19" extent="1-1"/>
 </signal>
 <signal name="OUT2">
@@
 <wire x1="-24.384" y1="68.834" x2="-24.384" y2="66.206" width="0.6096" layer="1"/>
 <wire x1="-24.384" y1="66.206" x2="-24.55" y2="66.04" width="0.6096" layer="1"/>
+<contactref element="U$1" pad="5"/>
+<wire x1="-23.13" y1="49.67" x2="-24.55" y2="66.04" width="0" layer="19" extent="1-1"/>
 </signal>
 <signal name="OUT3">
@@
 <wire x1="15.24" y1="68.58" x2="17.78" y2="66.04" width="0.6096" layer="1"/>
 <wire x1="17.78" y1="66.04" x2="19.05" y2="66.04" width="0.6096" layer="1"/>
+<contactref element="U$1" pad="6"/>
+<wire x1="-23.13" y1="54.47" x2="1.27" y2="59.69" width="0" layer="19" extent="1-1"/>
 </signal>
 <signal name="OUT4">
@@
 <wire x1="3.39" y1="66.04" x2="3.39" y2="68.668" width="0.6096" layer="1"/>
 <wire x1="3.39" y1="68.668" x2="3.556" y2="68.834" width="0.6096" layer="1"/>
+<contactref element="U$1" pad="7"/>
+<wire x1="-23.63" y1="54.47" x2="1.27" y2="57.15" width="0" layer="19" extent="1-1"/>
 </signal>
 <signal name="N$2">
@@
 <wire x1="-12.7" y1="69.59869375" x2="-12.7" y2="67.31" width="0.6096" layer="1"/>
 </signal>
+<signal name="N$1">
+<contactref element="U$1" pad="1"/>
+<contactref element="R13" pad="1"/>
+<wire x1="-41.91" y1="45.72" x2="-25.13" y2="49.67" width="0" layer="19" extent="1-1"/>
+</signal>
+<signal name="N$7">
+<contactref element="U$1" pad="2"/>
+<contactref element="R14" pad="2"/>
+<wire x1="-24.63" y1="49.67" x2="-34.29" y2="39.37" width="0" layer="19" extent="1-1"/>
+</signal>
+<signal name="N$6">
+<contactref element="U$1" pad="9"/>
+<contactref element="R16" pad="2"/>
+<wire x1="-24.63" y1="54.47" x2="-34.29" y2="49.53" width="0" layer="19" extent="1-1"/>
+</signal>
+<signal name="N$8">
+<contactref element="U$1" pad="10"/>
+<contactref element="R15" pad="2"/>
+<wire x1="-25.13" y1="54.47" x2="-30.48" y2="34.29" width="0" layer="19" extent="1-1"/>
+</signal>
 </signals>

Commit message: modifiche
Parts:
- moved R14 54.9 mm to (7.62, 69.8), turned to 90 degrees
- moved R16 54.7 mm to (12.7, 69.8), turned to 90 degrees
- moved R13 54.0 mm to (10.2, 69.8), turned to 90 degrees
- moved R15 40.3 mm to (-15.2, 69.8), turned to 90 degrees
- moved C5 33.8 mm to (0.00, 63.5)
- moved R7 27.4 mm to (0.00, 43.2), turned to 0 degrees
- moved U$1 25.3 mm to (0.00, 59.7), turned to 270 degrees
- moved R5 6.35 mm to (15.2, 69.8)
- moved R8 5.68 mm to (-11.4, 69.8), turned to 90 degrees
- moved R6 3.81 mm to (17.8, 69.8)
- moved R2 3.59 mm to (-19.1, 69.8), turned to 270 degrees
- moved R1 2.54 mm to (-7.62, 69.8)
- moved SV1 2.54 mm to (0.00, 54.6), turned to 180 degrees
- moved R3 1.27 mm to (20.3, 69.8)
- turned D7 to 90 degrees
Connections:
- removed net N$1: R13.1, U$1.1
- removed net N$6: R16.2, U$1.9
- removed net N$7: R14.2, U$1.2
- removed net N$8: R15.2, U$1.10
- new net ADDR: R13.1, SV1.3, U$1.1
- new net ALERT: R14.2, SV1.5, U$1.2
- new net SCL: R15.2, SV1.2, U$1.10
- new net SDA: R16.2, SV1.4, U$1.9
- net OUT1: no longer SV1.4
- net OUT2: no longer SV1.2
- net OUT3: no longer SV1.5
- net OUT4: no longer SV1.3
Routing:
- net ALERT: track 0.00 -> 39.6 mm, vias 0 -> 2
- net VCC: track 100.5 -> 138.9 mm, vias 0 -> 4
- net OUT2: track 43.7 -> 14.9 mm, vias 3 -> 0
- net ADDR: track 0.00 -> 19.8 mm
- net N$4: track 20.1 -> 3.07 mm
- net SCL: track 0.00 -> 10.7 mm
- net OUT1: track 43.6 -> 35.9 mm, vias 0 -> 1
- net OUT4: track 57.2 -> 50.0 mm, vias 1 -> 2
- net N$3: track 14.3 -> 10.5 mm
- net N$2: track 18.6 -> 22.0 mm, vias 1 -> 2
- net OUT3: track 40.9 -> 42.5 mm, vias 1 -> 2

Commit message: modiche 2
Parts:
- turned R5 to 270 degrees
- turned R6 to 270 degrees
- turned R8 to 270 degrees
Routing:
- net N$3: track 10.5 -> 18.4 mm, vias 0 -> 2
- net VCC: track 138.9 -> 145.6 mm
- net N$2: track 22.0 -> 20.9 mm, vias 2 -> 0
Changed lines of the file:
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@@
 <element name="R3" library="resistor" library_urn="urn:adsk.eagle:library:348" package="0204/7" package3d_urn="urn:adsk.eagle:package:25945/1" value="" x="20.32" y="69.85" rot="R270"/>
 <element name="R4" library="resistor" library_urn="urn:adsk.eagle:library:348" package="0204/7" package3d_urn="urn:adsk.eagle:package:25945/1" value="" x="35.56" y="69.85" rot="R270"/>
-<element name="R5" library="rcl" library_urn="urn:adsk.eagle:library:334" package="0204/7" package3d_urn="urn:adsk.eagle:package:23498/1" value="" x="15.24" y="69.85" rot="R90"/>
-<element name="R6" library="rcl" library_urn="urn:adsk.eagle:library:334" package="0204/7" package3d_urn="urn:adsk.eagle:package:23498/1" value="" x="17.78" y="69.85" rot="R90"/>
+<element name="R5" library="rcl" library_urn="urn:adsk.eagle:library:334" package="0204/7" package3d_urn="urn:adsk.eagle:package:23498/1" value="" x="15.24" y="69.85" rot="R270"/>
+<element name="R6" library="rcl" library_urn="urn:adsk.eagle:library:334" package="0204/7" package3d_urn="urn:adsk.eagle:package:23498/1" value="" x="17.78" y="69.85" rot="R270"/>
 <element name="R7" library="rcl" library_urn="urn:adsk.eagle:library:334" package="0204/7" package3d_urn="urn:adsk.eagle:package:23498/1" value="" x="0" y="43.18"/>
-<element name="R8" library="rcl" library_urn="urn:adsk.eagle:library:334" package="0204/7" package3d_urn="urn:adsk.eagle:package:23498/1" value="" x="-11.43" y="69.85" rot="R90"/>
+<element name="R8" library="rcl" library_urn="urn:adsk.eagle:library:334" package="0204/7" package3d_urn="urn:adsk.eagle:package:23498/1" value="" x="-11.43" y="69.85" rot="R270"/>
 <element name="SV1" library="con-lstb" library_urn="urn:adsk.eagle:library:162" package="MA03-2" package3d_urn="urn:adsk.eagle:package:8334/1" value="" x="0" y="54.61" rot="R180">
 <attribute name="MF" value="" x="0" y="54.61" size="1.778" layer="27" rot="R180" display="off"/>
@@
 <wire x1="8.89" y1="68.58" x2="11.43" y2="68.58" width="0.6096" layer="16"/>
 <wire x1="12.7" y1="67.31" x2="11.43" y2="68.58" width="0.6096" layer="16"/>
-<wire x1="15.24" y1="73.66" x2="17.78" y2="73.66" width="0.6096" layer="16"/>
-<wire x1="17.78" y1="73.66" x2="17.78" y2="71.12" width="0.6096" layer="16"/>
-<wire x1="17.78" y1="71.12" x2="19.05" y2="69.85" width="0.6096" layer="16"/>
 <wire x1="19.05" y1="69.85" x2="21.59" y2="69.85" width="0.6096" layer="16"/>
 <wire x1="21.59" y1="69.85" x2="22.86" y2="71.12" width="0.6096" layer="16"/>
@@
 <wire x1="5.08" y1="72.39" x2="2.54" y2="72.39" width="0.6096" layer="16"/>
 <wire x1="1.524" y1="70.866" x2="1.524" y2="72.136" width="0.6096" layer="16"/>
-<wire x1="1.524" y1="72.136" x2="0" y2="73.66" width="0.6096" layer="16"/>
+<wire x1="0" y1="73.66" x2="1.524" y2="72.136" width="0.6096" layer="16"/>
 <wire x1="-7.62" y1="71.12" x2="-11.43" y2="71.12" width="0.6096" layer="16"/>
 <wire x1="12.7" y1="66.04" x2="12.7" y2="67.31" width="0.6096" layer="16"/>
-<wire x1="12.7" y1="67.31" x2="16.51" y2="71.12" width="0.6096" layer="16"/>
-<wire x1="16.51" y1="71.12" x2="17.78" y2="71.12" width="0.6096" layer="16"/>
 <wire x1="1.524" y1="48.006" x2="1.27" y2="48.26" width="0.6096" layer="16"/>
 <wire x1="1.27" y1="48.26" x2="-2.54" y2="52.07" width="0.6096" layer="16"/>
@@
 <wire x1="-11.43" y1="71.12" x2="-13.335" y2="69.215" width="0.6096" layer="16"/>
 <wire x1="-13.335" y1="69.215" x2="-14.605" y2="69.215" width="0.6096" layer="16"/>
-<wire x1="-11.43" y1="71.12" x2="-11.43" y2="73.66" width="0.6096" layer="16"/>
+<wire x1="-11.43" y1="68.58" x2="-12.065" y2="69.215" width="0.6096" layer="16"/>
+<wire x1="-12.065" y1="69.215" x2="-13.335" y2="69.215" width="0.6096" layer="16"/>
+<wire x1="-11.43" y1="66.04" x2="-11.43" y2="68.58" width="0.6096" layer="16"/>
+<wire x1="12.7" y1="66.04" x2="15.24" y2="66.04" width="0.6096" layer="16"/>
+<wire x1="15.24" y1="66.04" x2="17.78" y2="66.04" width="0.6096" layer="16"/>
+<wire x1="17.78" y1="66.04" x2="17.78" y2="68.58" width="0.6096" layer="16"/>
+<wire x1="17.78" y1="68.58" x2="19.05" y2="69.85" width="0.6096" layer="16"/>
+<wire x1="-7.62" y1="71.12" x2="-5.08" y2="73.66" width="0.6096" layer="16"/>
+<wire x1="-5.08" y1="73.66" x2="0" y2="73.66" width="0.6096" layer="16"/>
 </signal>
 <signal name="OUT1">
@@
 <wire x1="0" y1="73.66" x2="5.08" y2="73.66" width="0.6096" layer="1"/>
 <wire x1="5.08" y1="73.66" x2="7.62" y2="71.12" width="0.6096" layer="1"/>
-<wire x1="7.62" y1="71.12" x2="10.16" y2="71.12" width="0.6096" layer="1"/>
-<via x="10.16" y="71.12" extent="1-16" drill="0.35"/>
-<wire x1="10.16" y1="71.12" x2="12.7" y2="68.58" width="0.6096" layer="16"/>
-<via x="12.7" y="68.58" extent="1-16" drill="0.35"/>
-<wire x1="12.7" y1="68.58" x2="15.24" y2="66.04" width="0.6096" layer="1"/>
+<wire x1="7.62" y1="71.12" x2="12.7" y2="71.12" width="0.6096" layer="1"/>
+<wire x1="12.7" y1="71.12" x2="15.24" y2="73.66" width="0.6096" layer="1"/>
 </signal>
 <signal name="N$3">
 <contactref element="R6" pad="1"/>
 <contactref element="D6" pad="A"/>
-<wire x1="24.13" y1="67.31" x2="19.05" y2="67.31" width="0.6096" layer="16"/>
-<wire x1="19.05" y1="67.31" x2="17.78" y2="66.04" width="0.6096" layer="16"/>
 <wire x1="26.67" y1="69.85" x2="24.13" y2="67.31" width="0.6096" layer="16"/>
+<wire x1="24.13" y1="67.31" x2="21.59" y2="67.31" width="0.6096" layer="16"/>
+<wire x1="21.59" y1="67.31" x2="20.32" y2="68.58" width="0.6096" layer="16"/>
+<via x="20.32" y="68.58" extent="1-16" drill="0.35"/>
+<wire x1="20.32" y1="68.58" x2="16.51" y2="68.58" width="0.6096" layer="1"/>
+<via x="16.51" y="68.58" extent="1-16" drill="0.35"/>
+<wire x1="16.51" y1="68.58" x2="15.24" y2="69.85" width="0.6096" layer="16"/>
+<wire x1="15.24" y1="69.85" x2="15.24" y2="71.12" width="0.6096" layer="16"/>
+<wire x1="15.24" y1="71.12" x2="17.78" y2="73.66" width="0.6096" layer="16"/>
 </signal>
 <signal name="N$4">
@@
 <wire x1="-29.21" y1="72.39" x2="-20.32" y2="72.39" width="0.6096" layer="1"/>
 <wire x1="-20.32" y1="72.39" x2="-17.78" y2="69.85" width="0.6096" layer="1"/>
-<wire x1="-12.7" y1="69.85" x2="-11.43" y2="68.58" width="0.6096" layer="1"/>
-<wire x1="-11.43" y1="68.58" x2="-11.43" y2="66.04" width="0.6096" layer="1"/>
 <wire x1="-17.78" y1="69.85" x2="-12.7" y2="69.85" width="0.6096" layer="1"/>
+<wire x1="-12.7" y1="69.85" x2="-11.43" y2="71.12" width="0.6096" layer="1"/>
+<wire x1="-11.43" y1="71.12" x2="-11.43" y2="73.66" width="0.6096" layer="1"/>
 </signal>
 <signal name="ADDR">
@@
 <contactref element="R16" pad="2"/>
 <contactref element="SV1" pad="4"/>
-<wire x1="2.4" y1="60.19" x2="12.7" y2="73.66" width="0" layer="19" extent="1-1"/>
+<wire x1="2.4" y1="60.19" x2="3.4168" y2="60.19" width="0" layer="19" extent="1-16"/>
+<wire x1="3.4168" y1="60.19" x2="3.81" y2="59.7968" width="0" layer="19" extent="1-16"/>
+<wire x1="3.81" y1="59.7968" x2="4.3476" y2="59.7968" width="0" layer="19" extent="1-16"/>
+<wire x1="4.3476" y1="59.7968" x2="4.4544" y2="59.69" width="0" layer="19" extent="1-16"/>
+<wire x1="4.3476" y1="59.7968" x2="12.7" y2="73.66" width="0" layer="19" extent="1-1"/>
 <wire x1="0" y1="53.34" x2="2.4" y2="60.19" width="0" layer="19" extent="1-1"/>
 </signal>
