File: hardware/electronics/sensori-linea/sensore-linea.brd (EAGLE design)
At the start: 88.1 x 42 mm, 27 parts, among them T1 BP103, T2 BP103, T3 BP103, T4 BP103

Commit message: base
Parts:
- moved C2 2.01 mm to (27.3, 66.7), turned to 90 degrees
Routing:
- net GND: track 1.45 -> 16.0 mm, vias 4 -> 5
- net ALERT: track 33.8 -> 38.0 mm
- net VCC: track 119.8 -> 116.4 mm, vias 3 -> 5
- net SDA: track 36.4 -> 33.8 mm
- net OUT3: track 45.2 -> 43.7 mm
- net N$3: track 18.4 -> 19.2 mm
- net ADDR: track 19.9 -> 20.7 mm
- net SCL: track 39.2 -> 38.6 mm
