File: hardware/electronics/Base/base.brd (EAGLE design)
At the start: 160 x 100 mm, 25 parts, among them IC1 7805T, IC2 74LS595D, IC3 74LS595D

Commit message: aggiornamenti
Parts:
- removed B1: SD_MMC_CARDSD_PCB, SparkFun-Boards:SD-MMC-CARD
Changed lines of the file:
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@@
 </element>
 <element name="IC3" library="74xx-us" library_urn="urn:adsk.eagle:library:88" package="SO16" package3d_urn="urn:adsk.eagle:package:2918/1" value="74LS595D" x="-142.24" y="-266.7"/>
-<element name="B1" library="SparkFun-Boards" package="SD-MMC-CARD" value="SD_MMC_CARDSD_PCB" x="-161.29" y="-257.81"/>
 </elements>
 <signals>
