File: hardware/electronics/Base/base.brd (EAGLE design)
At the start: 160 x 100 mm, 19 parts, among them IC1 7805T, IC2 74LS595D

Commit message: base
Parts:
- added X1, X2, X3, X4: (no value), con-wago-500:W237-102
Connections:
- net MOT1_INA renamed MOT1-INA
- net MOT1_INB renamed MOT1-INB
- net MOT2_INA renamed MOT2-INA
- net MOT2_INB renamed MOT2-INB
- net MOT3_INA renamed MOT3-INA
- net MOT3_INB renamed MOT3-INB
- net MOT4_INA renamed MOT4-INA
- net MOT4_INB renamed MOT4-INB
- new net CLOCK: IC2.11, U$2.27
- new net DATA-IN: IC2.14, U$2.28
- new net LATCH: IC2.12, U$2.26
- new net MOT1-PWM: U$3.PWM
- new net MOT2-PWM: U$5.PWM
- new net MOT3-PWM: U$4.PWM
- new net MOT4-PWM: U$7.PWM
- net MOT1_PWM: no longer U$3.PWM
- net MOT2_PWM: no longer U$5.PWM
- net MOT3_PWM: no longer U$4.PWM
- net MOT4_PWM: no longer U$7.PWM
Changed lines of the file:
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@@
 <attribute name="MOTOR" value="motor" x="-59.69" y="-170.18" size="1.778" layer="27" display="off"/>
+</element>
+<element name="X1" library="con-wago-500" library_urn="urn:adsk.eagle:library:195" package="W237-102" package3d_urn="urn:adsk.eagle:package:10688/1" value="" x="-68.58" y="-205.74">
+<attribute name="MF" value="" x="-68.58" y="-205.74" size="1.778" layer="27" display="off"/>
+<attribute name="MPN" value="237-102" x="-68.58" y="-205.74" size="1.778" layer="27" display="off"/>
+<attribute name="OC_FARNELL" value="unknown" x="-68.58" y="-205.74" size="1.778" layer="27" display="off"/>
+<attribute name="OC_NEWARK" value="70K9898" x="-68.58" y="-205.74" size="1.778" layer="27" display="off"/>
+</element>
+<element name="X2" library="con-wago-500" library_urn="urn:adsk.eagle:library:195" package="W237-102" package3d_urn="urn:adsk.eagle:package:10688/1" value="" x="-68.58" y="-224.79">
+<attribute name="MF" value="" x="-68.58" y="-224.79" size="1.778" layer="27" display="off"/>
+<attribute name="MPN" value="237-102" x="-68.58" y="-224.79" size="1.778" layer="27" display="off"/>
+<attribute name="OC_FARNELL" value="unknown" x="-68.58" y="-224.79" size="1.778" layer="27" display="off"/>
+<attribute name="OC_NEWARK" value="70K9898" x="-68.58" y="-224.79" size="1.778" layer="27" display="off"/>
+</element>
+<element name="X3" library="con-wago-500" library_urn="urn:adsk.eagle:library:195" package="W237-102" package3d_urn="urn:adsk.eagle:package:10688/1" value="" x="-68.58" y="-243.84">
+<attribute name="MF" value="" x="-68.58" y="-243.84" size="1.778" layer="27" display="off"/>
+<attribute name="MPN" value="237-102" x="-68.58" y="-243.84" size="1.778" layer="27" display="off"/>
+<attribute name="OC_FARNELL" value="unknown" x="-68.58" y="-243.84" size="1.778" layer="27" display="off"/>
+<attribute name="OC_NEWARK" value="70K9898" x="-68.58" y="-243.84" size="1.778" layer="27" display="off"/>
+</element>
+<element name="X4" library="con-wago-500" library_urn="urn:adsk.eagle:library:195" package="W237-102" package3d_urn="urn:adsk.eagle:package:10688/1" value="" x="-68.58" y="-262.89">
+<attribute name="MF" value="" x="-68.58" y="-262.89" size="1.778" layer="27" display="off"/>
+<attribute name="MPN" value="237-102" x="-68.58" y="-262.89" size="1.778" layer="27" display="off"/>
+<attribute name="OC_FARNELL" value="unknown" x="-68.58" y="-262.89" size="1.778" layer="27" display="off"/>
+<attribute name="OC_NEWARK" value="70K9898" x="-68.58" y="-262.89" size="1.778" layer="27" display="off"/>
 </element>
 </elements>
@@
 <contactref element="U$3" pad="GNDMOT-1"/>
 </signal>
-<signal name="MOT1_INB">
+<signal name="MOT1-INB">
 <contactref element="U$3" pad="INB"/>
 </signal>
@@
 <signal name="MOT1_PWM">
 <contactref element="U$2" pad="5"/>
-<contactref element="U$3" pad="PWM"/>
-<wire x1="-45.72" y1="20.32" x2="-15.24" y2="45.72" width="0" layer="19" extent="1-1"/>
 </signal>
 <signal name="MOT2_PWM">
 <contactref element="U$2" pad="6"/>
-<contactref element="U$5" pad="PWM"/>
-<wire x1="-45.72" y1="17.78" x2="-30.48" y2="-81.28" width="0" layer="19" extent="1-1"/>
 </signal>
 <signal name="MOT3_PWM">
 <contactref element="U$2" pad="25"/>
-<contactref element="U$4" pad="PWM"/>
-<wire x1="-38.1" y1="12.7" x2="-30.48" y2="-33.02" width="0" layer="19" extent="1-1"/>
 </signal>
 <signal name="MOT4_PWM">
 <contactref element="U$2" pad="32"/>
+</signal>
+<signal name="LATCH">
+<contactref element="IC2" pad="12"/>
+<contactref element="U$2" pad="26"/>
+<wire x1="-38.1" y1="10.16" x2="-18.415" y2="91.9734" width="0" layer="19" extent="1-1"/>
+</signal>
+<signal name="CLOCK">
+<contactref element="IC2" pad="11"/>
+<contactref element="U$2" pad="27"/>
+<wire x1="-38.1" y1="7.62" x2="-17.145" y2="91.9734" width="0" layer="19" extent="1-1"/>
+</signal>
+<signal name="DATA-IN">
+<contactref element="IC2" pad="14"/>
+<contactref element="U$2" pad="28"/>
+<wire x1="-38.1" y1="5.08" x2="-20.955" y2="91.9734" width="0" layer="19" extent="1-1"/>
+</signal>
+<signal name="MOT1-PWM">
+<contactref element="U$3" pad="PWM"/>
+</signal>
+<signal name="MOT1-INA">
+<contactref element="U$3" pad="INA"/>
+<contactref element="IC2" pad="15"/>
+<wire x1="-15.24" y1="40.64" x2="-22.225" y2="91.9734" width="0" layer="19" extent="1-1"/>
+</signal>
+<signal name="MOT3-INB">
+<contactref element="U$4" pad="INB"/>
+<contactref element="IC2" pad="5"/>
+<wire x1="-30.48" y1="-25.4" x2="-18.415" y2="85.8266" width="0" layer="19" extent="1-1"/>
+</signal>
+<signal name="MOT3-PWM">
+<contactref element="U$4" pad="PWM"/>
+</signal>
+<signal name="MOT3-INA">
+<contactref element="U$4" pad="INA"/>
+<contactref element="IC2" pad="4"/>
+<wire x1="-19.685" y1="85.8266" x2="-30.48" y2="-38.1" width="0" layer="19" extent="1-1"/>
+</signal>
+<signal name="MOT4-INA">
+<contactref element="U$7" pad="INA"/>
+<contactref element="IC2" pad="6"/>
+<wire x1="-17.145" y1="85.8266" x2="-30.48" y2="-182.88" width="0" layer="19" extent="1-1"/>
+</signal>
+<signal name="MOT4-PWM">
 <contactref element="U$7" pad="PWM"/>
-<wire x1="-35.56" y1="12.7" x2="-30.48" y2="-177.8" width="0" layer="19" extent="1-1"/>
-</signal>
-<signal name="MOT1_INA">
-<contactref element="IC2" pad="15"/>
-<contactref element="U$3" pad="INA"/>
-<wire x1="-15.24" y1="40.64" x2="-22.225" y2="91.9734" width="0" layer="19" extent="1-1"/>
-</signal>
-<signal name="MOT2_INB">
+</signal>
+<signal name="MOT4-INB">
+<contactref element="U$7" pad="INB"/>
+<contactref element="IC2" pad="7"/>
+<wire x1="-15.875" y1="85.8266" x2="-30.48" y2="-170.18" width="0" layer="19" extent="1-1"/>
+</signal>
+<signal name="MOT2-INA">
+<contactref element="U$5" pad="INA"/>
+<contactref element="IC2" pad="2"/>
+<wire x1="-22.225" y1="85.8266" x2="-30.48" y2="-86.36" width="0" layer="19" extent="1-1"/>
+</signal>
+<signal name="MOT2-PWM">
+<contactref element="U$5" pad="PWM"/>
+</signal>
+<signal name="MOT2-INB">
+<contactref element="U$5" pad="INB"/>
 <contactref element="IC2" pad="1"/>
 <contactref element="IC2" pad="3"/>
-<contactref element="U$5" pad="INB"/>
 <wire x1="-23.495" y1="85.8266" x2="-30.48" y2="-73.66" width="0" layer="19" extent="1-1"/>
 <wire x1="-20.955" y1="85.8266" x2="-23.495" y2="85.8266" width="0" layer="19" extent="1-1"/>
 </signal>
-<signal name="MOT2_INA">
-<contactref element="IC2" pad="2"/>
-<contactref element="U$5" pad="INA"/>
-<wire x1="-22.225" y1="85.8266" x2="-30.48" y2="-86.36" width="0" layer="19" extent="1-1"/>
-</signal>
-<signal name="MOT3_INA">
-<contactref element="IC2" pad="4"/>
-<contactref element="U$4" pad="INA"/>
-<wire x1="-19.685" y1="85.8266" x2="-30.48" y2="-38.1" width="0" layer="19" extent="1-1"/>
-</signal>
-<signal name="MOT3_INB">
-<contactref element="IC2" pad="5"/>
-<contactref element="U$4" pad="INB"/>
-<wire x1="-30.48" y1="-25.4" x2="-18.415" y2="85.8266" width="0" layer="19" extent="1-1"/>
-</signal>
-<signal name="MOT4_INA">
-<contactref element="IC2" pad="6"/>
-<contactref element="U$7" pad="INA"/>
-<wire x1="-17.145" y1="85.8266" x2="-30.48" y2="-182.88" width="0" layer="19" extent="1-1"/>
-</signal>
-<signal name="MOT4_INB">
-<contactref element="IC2" pad="7"/>
-<contactref element="U$7" pad="INB"/>
-<wire x1="-15.875" y1="85.8266" x2="-30.48" y2="-170.18" width="0" layer="19" extent="1-1"/>
-</signal>
 </signals>

Commit message: base
Parts:
- moved X1 81.8 mm to (-124.5, -146.1)
- moved X2 8.89 mm to (-59.7, -224.8)
Connections:
- new net MOTORE1-1: U$3.INMOT1, X1.1
- new net MOTORE1-2: U$3.INMOT2, X1.2
- new net MOTORE2-1: U$5.INMOT1, X2.1
- new net MOTORE2-2: U$5.INMOT2, X2.2
- new net MOTORE3-1: U$4.INMOT1, X3.1
- new net MOTORE3-2: U$4.INMOT2, X3.2
- new net MOTORE4-1: U$7.INMOT1, X4.1
- new net MOTORE4-2: U$7.INMOT2, X4.2
Changed lines of the file:
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@@
 <attribute name="MOTOR" value="motor" x="-59.69" y="-170.18" size="1.778" layer="27" display="off"/>
 </element>
-<element name="X1" library="con-wago-500" library_urn="urn:adsk.eagle:library:195" package="W237-102" package3d_urn="urn:adsk.eagle:package:10688/1" value="" x="-68.58" y="-205.74">
-<attribute name="MF" value="" x="-68.58" y="-205.74" size="1.778" layer="27" display="off"/>
-<attribute name="MPN" value="237-102" x="-68.58" y="-205.74" size="1.778" layer="27" display="off"/>
-<attribute name="OC_FARNELL" value="unknown" x="-68.58" y="-205.74" size="1.778" layer="27" display="off"/>
-<attribute name="OC_NEWARK" value="70K9898" x="-68.58" y="-205.74" size="1.778" layer="27" display="off"/>
-</element>
-<element name="X2" library="con-wago-500" library_urn="urn:adsk.eagle:library:195" package="W237-102" package3d_urn="urn:adsk.eagle:package:10688/1" value="" x="-68.58" y="-224.79">
-<attribute name="MF" value="" x="-68.58" y="-224.79" size="1.778" layer="27" display="off"/>
-<attribute name="MPN" value="237-102" x="-68.58" y="-224.79" size="1.778" layer="27" display="off"/>
-<attribute name="OC_FARNELL" value="unknown" x="-68.58" y="-224.79" size="1.778" layer="27" display="off"/>
-<attribute name="OC_NEWARK" value="70K9898" x="-68.58" y="-224.79" size="1.778" layer="27" display="off"/>
+<element name="X1" library="con-wago-500" library_urn="urn:adsk.eagle:library:195" package="W237-102" package3d_urn="urn:adsk.eagle:package:10688/1" value="" x="-124.46" y="-146.05">
+<attribute name="MF" value="" x="-124.46" y="-146.05" size="1.778" layer="27" display="off"/>
+<attribute name="MPN" value="237-102" x="-124.46" y="-146.05" size="1.778" layer="27" display="off"/>
+<attribute name="OC_FARNELL" value="unknown" x="-124.46" y="-146.05" size="1.778" layer="27" display="off"/>
+<attribute name="OC_NEWARK" value="70K9898" x="-124.46" y="-146.05" size="1.778" layer="27" display="off"/>
+</element>
+<element name="X2" library="con-wago-500" library_urn="urn:adsk.eagle:library:195" package="W237-102" package3d_urn="urn:adsk.eagle:package:10688/1" value="" x="-59.69" y="-224.79">
+<attribute name="MF" value="" x="-59.69" y="-224.79" size="1.778" layer="27" display="off"/>
+<attribute name="MPN" value="237-102" x="-59.69" y="-224.79" size="1.778" layer="27" display="off"/>
+<attribute name="OC_FARNELL" value="unknown" x="-59.69" y="-224.79" size="1.778" layer="27" display="off"/>
+<attribute name="OC_NEWARK" value="70K9898" x="-59.69" y="-224.79" size="1.778" layer="27" display="off"/>
 </element>
 <element name="X3" library="con-wago-500" library_urn="urn:adsk.eagle:library:195" package="W237-102" package3d_urn="urn:adsk.eagle:package:10688/1" value="" x="-68.58" y="-243.84">
@@
 <wire x1="-20.955" y1="85.8266" x2="-23.495" y2="85.8266" width="0" layer="19" extent="1-1"/>
 </signal>
+<signal name="MOTORE1-2">
+<contactref element="U$3" pad="INMOT2"/>
+<contactref element="X1" pad="2"/>
+<wire x1="-49.53" y1="41.91" x2="-121.96" y2="-147.32" width="0" layer="19" extent="1-1"/>
+</signal>
+<signal name="MOTORE3-1">
+<contactref element="U$4" pad="INMOT1"/>
+<contactref element="X3" pad="1"/>
+<wire x1="-71.08" y1="-245.11" x2="-64.77" y2="-31.75" width="0" layer="19" extent="1-1"/>
+</signal>
+<signal name="MOTORE3-2">
+<contactref element="U$4" pad="INMOT2"/>
+<contactref element="X3" pad="2"/>
+<wire x1="-66.08" y1="-245.11" x2="-64.77" y2="-36.83" width="0" layer="19" extent="1-1"/>
+</signal>
+<signal name="MOTORE2-2">
+<contactref element="U$5" pad="INMOT2"/>
+<contactref element="X2" pad="2"/>
+<wire x1="-57.19" y1="-226.06" x2="-64.77" y2="-85.09" width="0" layer="19" extent="1-1"/>
+</signal>
+<signal name="MOTORE1-1">
+<contactref element="X1" pad="1"/>
+<contactref element="U$3" pad="INMOT1"/>
+<wire x1="-49.53" y1="46.99" x2="-126.96" y2="-147.32" width="0" layer="19" extent="1-1"/>
+</signal>
+<signal name="MOTORE4-2">
+<contactref element="X4" pad="2"/>
+<contactref element="U$7" pad="INMOT2"/>
+<wire x1="-66.08" y1="-264.16" x2="-64.77" y2="-181.61" width="0" layer="19" extent="1-1"/>
+</signal>
+<signal name="MOTORE4-1">
+<contactref element="X4" pad="1"/>
+<contactref element="U$7" pad="INMOT1"/>
+<wire x1="-71.08" y1="-264.16" x2="-64.77" y2="-176.53" width="0" layer="19" extent="1-1"/>
+</signal>
+<signal name="MOTORE2-1">
+<contactref element="X2" pad="1"/>
+<contactref element="U$5" pad="INMOT1"/>
+<wire x1="-62.19" y1="-226.06" x2="-64.77" y2="-80.01" width="0" layer="19" extent="1-1"/>
+</signal>
 </signals>

Commit message: base
Parts:
- added B1: SD_MMC_CARDSD_PCB, SparkFun-Boards:SD-MMC-CARD
- added IC3: 74LS595D, 74xx-us:SO16
Connections:
- new net VCC: IC3.16
- net GND: now also IC3.8
Changed lines of the file:
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@@
 <attribute name="OC_NEWARK" value="70K9898" x="-68.58" y="-262.89" size="1.778" layer="27" display="off"/>
 </element>
+<element name="IC3" library="74xx-us" library_urn="urn:adsk.eagle:library:88" package="SO16" package3d_urn="urn:adsk.eagle:package:2918/1" value="74LS595D" x="-142.24" y="-266.7"/>
+<element name="B1" library="SparkFun-Boards" package="SD-MMC-CARD" value="SD_MMC_CARDSD_PCB" x="-161.29" y="-257.81"/>
 </elements>
 <signals>
@@
 <contactref element="U$7" pad="GNDMOT-1"/>
 <contactref element="IC2" pad="13"/>
+<contactref element="IC3" pad="8"/>
 <wire x1="-30.48" y1="-165.1" x2="-64.77" y2="-171.45" width="0" layer="19" extent="1-1"/>
 <wire x1="-30.48" y1="-160.02" x2="-30.48" y2="-165.1" width="0" layer="19" extent="1-1"/>
@@
 <wire x1="-19.685" y1="91.9734" x2="-29.08" y2="87.63" width="0" layer="19" extent="1-1"/>
 <wire x1="-14.605" y1="85.8266" x2="-19.685" y2="91.9734" width="0" layer="19" extent="1-1"/>
+<wire x1="-137.795" y1="-269.7734" x2="-64.77" y2="-171.45" width="0" layer="19" extent="1-1"/>
 </signal>
 <signal name="VIN">
@@
 <wire x1="-62.19" y1="-226.06" x2="-64.77" y2="-80.01" width="0" layer="19" extent="1-1"/>
 </signal>
+<signal name="VCC">
+<contactref element="IC3" pad="16"/>
+</signal>
 </signals>

Commit message: aggiornamenti base
Parts:
- removed B1: SD_MMC_CARDSD_PCB, SparkFun-Boards:SD-MMC-CARD
- added DIS1: HD-H103, display-hp:HDSP-M
- added IC4: 74LS595D, 74xx-us:SO16
Connections:
- net DATA-IN renamed DATA-IN1
- removed net VCC: IC3.16
- new net N$10: IC4.14
- new net N$5: IC3.14
- net 3.3V: now also IC3.10, IC3.16, IC4.10, IC4.16
- net CLOCK: now also IC3.11, IC4.11
- net GND: now also IC3.13, IC4.13, IC4.8
- net LATCH: now also IC3.12, IC4.12
Changed lines of the file:
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@@
 </element>
 <element name="IC3" library="74xx-us" library_urn="urn:adsk.eagle:library:88" package="SO16" package3d_urn="urn:adsk.eagle:package:2918/1" value="74LS595D" x="-142.24" y="-266.7"/>
-<element name="B1" library="SparkFun-Boards" package="SD-MMC-CARD" value="SD_MMC_CARDSD_PCB" x="-161.29" y="-257.81"/>
+<element name="DIS1" library="display-hp" library_urn="urn:adsk.eagle:library:212" package="HDSP-M" package3d_urn="urn:adsk.eagle:package:13006/1" value="HD-H103" x="-161.29" y="-257.81">
+<attribute name="MF" value="" x="-161.29" y="-257.81" size="1.778" layer="27" display="off"/>
+<attribute name="MPN" value="" x="-161.29" y="-257.81" size="1.778" layer="27" display="off"/>
+<attribute name="OC_FARNELL" value="unknown" x="-161.29" y="-257.81" size="1.778" layer="27" display="off"/>
+<attribute name="OC_NEWARK" value="unknown" x="-161.29" y="-257.81" size="1.778" layer="27" display="off"/>
+</element>
+<element name="IC4" library="74xx-us" library_urn="urn:adsk.eagle:library:88" package="SO16" package3d_urn="urn:adsk.eagle:package:2918/1" value="74LS595D" x="-179.07" y="-266.7"/>
 </elements>
 <signals>
@@
 <contactref element="IC2" pad="13"/>
 <contactref element="IC3" pad="8"/>
+<contactref element="IC4" pad="8"/>
+<contactref element="IC3" pad="13"/>
+<contactref element="IC4" pad="13"/>
 <wire x1="-30.48" y1="-165.1" x2="-64.77" y2="-171.45" width="0" layer="19" extent="1-1"/>
 <wire x1="-30.48" y1="-160.02" x2="-30.48" y2="-165.1" width="0" layer="19" extent="1-1"/>
@@
 <wire x1="-19.685" y1="91.9734" x2="-29.08" y2="87.63" width="0" layer="19" extent="1-1"/>
 <wire x1="-14.605" y1="85.8266" x2="-19.685" y2="91.9734" width="0" layer="19" extent="1-1"/>
-<wire x1="-137.795" y1="-269.7734" x2="-64.77" y2="-171.45" width="0" layer="19" extent="1-1"/>
+<wire x1="-142.875" y1="-263.6266" x2="-64.77" y2="-171.45" width="0" layer="19" extent="1-1"/>
+<wire x1="-137.795" y1="-269.7734" x2="-142.875" y2="-263.6266" width="0" layer="19" extent="1-1"/>
+<wire x1="-174.625" y1="-269.7734" x2="-142.875" y2="-263.6266" width="0" layer="19" extent="1-1"/>
+<wire x1="-179.705" y1="-263.6266" x2="-174.625" y2="-269.7734" width="0" layer="19" extent="1-1"/>
 </signal>
 <signal name="VIN">
@@
 <contactref element="IC2" pad="16"/>
 <contactref element="IC2" pad="10"/>
+<contactref element="IC3" pad="16"/>
+<contactref element="IC4" pad="16"/>
+<contactref element="IC4" pad="10"/>
+<contactref element="IC3" pad="10"/>
+<wire x1="-175.895" y1="-263.6266" x2="-183.515" y2="-263.6266" width="0" layer="19" extent="1-1"/>
+<wire x1="-146.685" y1="-263.6266" x2="-175.895" y2="-263.6266" width="0" layer="19" extent="1-1"/>
+<wire x1="-139.065" y1="-263.6266" x2="-146.685" y2="-263.6266" width="0" layer="19" extent="1-1"/>
+<wire x1="-40.64" y1="2.54" x2="-139.065" y2="-263.6266" width="0" layer="19" extent="1-1"/>
+<wire x1="-35.56" y1="17.78" x2="-40.64" y2="2.54" width="0" layer="19" extent="1-1"/>
+<wire x1="-30.48" y1="30.48" x2="-35.56" y2="17.78" width="0" layer="19" extent="1-1"/>
+<wire x1="-15.24" y1="55.88" x2="-30.48" y2="30.48" width="0" layer="19" extent="1-1"/>
+<wire x1="-15.24" y1="72.39" x2="-15.24" y2="55.88" width="0" layer="19" extent="1-1"/>
+<wire x1="-15.875" y1="91.9734" x2="-15.24" y2="72.39" width="0" layer="19" extent="1-1"/>
 <wire x1="-23.495" y1="91.9734" x2="-15.875" y2="91.9734" width="0" layer="19" extent="1-1"/>
 <wire x1="-31.88" y1="87.63" x2="-23.495" y2="91.9734" width="0" layer="19" extent="1-1"/>
 <wire x1="-36.96" y1="87.63" x2="-31.88" y2="87.63" width="0" layer="19" extent="1-1"/>
 <wire x1="-45.72" y1="74.93" x2="-36.96" y2="87.63" width="0" layer="19" extent="1-1"/>
-<wire x1="-15.24" y1="72.39" x2="-15.875" y2="91.9734" width="0" layer="19" extent="1-1"/>
-<wire x1="-15.24" y1="55.88" x2="-15.24" y2="72.39" width="0" layer="19" extent="1-1"/>
-<wire x1="-30.48" y1="30.48" x2="-15.24" y2="55.88" width="0" layer="19" extent="1-1"/>
-<wire x1="-35.56" y1="17.78" x2="-30.48" y2="30.48" width="0" layer="19" extent="1-1"/>
-<wire x1="-40.64" y1="2.54" x2="-35.56" y2="17.78" width="0" layer="19" extent="1-1"/>
 </signal>
 <signal name="VBAT">
@@
 <contactref element="IC2" pad="12"/>
 <contactref element="U$2" pad="26"/>
-<wire x1="-38.1" y1="10.16" x2="-18.415" y2="91.9734" width="0" layer="19" extent="1-1"/>
+<contactref element="IC3" pad="12"/>
+<contactref element="IC4" pad="12"/>
+<wire x1="-141.605" y1="-263.6266" x2="-178.435" y2="-263.6266" width="0" layer="19" extent="1-1"/>
+<wire x1="-38.1" y1="10.16" x2="-141.605" y2="-263.6266" width="0" layer="19" extent="1-1"/>
+<wire x1="-18.415" y1="91.9734" x2="-38.1" y2="10.16" width="0" layer="19" extent="1-1"/>
 </signal>
 <signal name="CLOCK">
 <contactref element="IC2" pad="11"/>
 <contactref element="U$2" pad="27"/>
-<wire x1="-38.1" y1="7.62" x2="-17.145" y2="91.9734" width="0" layer="19" extent="1-1"/>
-</signal>
-<signal name="DATA-IN">
+<contactref element="IC3" pad="11"/>
+<contactref element="IC4" pad="11"/>
+<wire x1="-140.335" y1="-263.6266" x2="-177.165" y2="-263.6266" width="0" layer="19" extent="1-1"/>
+<wire x1="-38.1" y1="7.62" x2="-140.335" y2="-263.6266" width="0" layer="19" extent="1-1"/>
+<wire x1="-17.145" y1="91.9734" x2="-38.1" y2="7.62" width="0" layer="19" extent="1-1"/>
+</signal>
+<signal name="DATA-IN1">
 <contactref element="IC2" pad="14"/>
 <contactref element="U$2" pad="28"/>
@@
 <wire x1="-62.19" y1="-226.06" x2="-64.77" y2="-80.01" width="0" layer="19" extent="1-1"/>
 </signal>
-<signal name="VCC">
-<contactref element="IC3" pad="16"/>
+<signal name="N$5">
+<contactref element="IC3" pad="14"/>
+</signal>
+<signal name="N$10">
+<contactref element="IC4" pad="14"/>
 </signal>
 </signals>
