File: hardware/electronics/Base/base.brd (EAGLE design)
At the start: 160 x 100 mm, 26 parts, among them IC1 7805T, IC2 74LS595D, IC3 74LS595D, IC4 74LS595D

Commit message: schema base piu lbr
Parts:
- removed DIS1: HD-H103, display-hp:HDSP-M
- removed U$1: ALIM, Pololu switching alimentatore:ALIM_SWITCHING
- added U$6: REGOLATORE-3.3V-1A, libreria valerio:REGOLATORE-3.3V-1A
Connections:
- net 3.3V: now also U$6.VOUT; no longer U$1.VOUT
- net GND: no longer U$1.GND
- net N$1: now also U$6.VIN; no longer U$1.SHDN, U$1.VIN
Changed lines of the file:
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@@
 <element name="R1" library="resistor" library_urn="urn:adsk.eagle:library:348" package="M1206" package3d_urn="urn:adsk.eagle:package:26088/1" value="1K" x="-35.56" y="87.63"/>
 <element name="R2" library="resistor" library_urn="urn:adsk.eagle:library:348" package="M1206" package3d_urn="urn:adsk.eagle:package:26088/1" value="1K" x="-40.64" y="87.63"/>
-<element name="U$1" library="Pololu switching alimentatore" package="ALIM_SWITCHING" value="ALIM" x="-19.05" y="76.2">
-<attribute name="POLOLU" value="" x="-19.05" y="76.2" size="1.778" layer="27" display="off"/>
-</element>
 <element name="U$2" library="Teensy_3_and_LC_Series_Boards_v1.4" package="TEENSY_3.0-3.2_ALL_PINS_&amp;_PADS" value="TEENSY_3.1-3.2_ALL_PINS&amp;PADS" x="-38.1" y="19.05"/>
 <element name="U$3" library="VHN5019" package="MOTOR-SHIELD" value="VHN5019" x="-44.45" y="53.34">
@@
 </element>
 <element name="IC3" library="74xx-us" library_urn="urn:adsk.eagle:library:88" package="SO16" package3d_urn="urn:adsk.eagle:package:2918/1" value="74LS595D" x="-142.24" y="-266.7"/>
-<element name="DIS1" library="display-hp" library_urn="urn:adsk.eagle:library:212" package="HDSP-M" package3d_urn="urn:adsk.eagle:package:13006/1" value="HD-H103" x="-161.29" y="-257.81">
-<attribute name="MF" value="" x="-161.29" y="-257.81" size="1.778" layer="27" display="off"/>
-<attribute name="MPN" value="" x="-161.29" y="-257.81" size="1.778" layer="27" display="off"/>
-<attribute name="OC_FARNELL" value="unknown" x="-161.29" y="-257.81" size="1.778" layer="27" display="off"/>
-<attribute name="OC_NEWARK" value="unknown" x="-161.29" y="-257.81" size="1.778" layer="27" display="off"/>
-</element>
 <element name="IC4" library="74xx-us" library_urn="urn:adsk.eagle:library:88" package="SO16" package3d_urn="urn:adsk.eagle:package:2918/1" value="74LS595D" x="-179.07" y="-266.7"/>
+<element name="U$6" library="libreria valerio" package="REGOLATORE-3.3V-1A" value="REGOLATORE-3.3V-1A" x="-179.07" y="-292.1"/>
 </elements>
 <signals>
@@
 <contactref element="IC2" pad="8"/>
 <contactref element="C1" pad="-"/>
-<contactref element="U$1" pad="GND"/>
 <contactref element="D2" pad="C"/>
 <contactref element="C3" pad="2"/>
@@
 <wire x1="-40.64" y1="74.93" x2="-52.07" y2="74.93" width="0" layer="19" extent="1-1"/>
 <wire x1="-29.21" y1="74.93" x2="-40.64" y2="74.93" width="0" layer="19" extent="1-1"/>
-<wire x1="-17.78" y1="72.39" x2="-29.21" y2="74.93" width="0" layer="19" extent="1-1"/>
 <wire x1="-29.08" y1="87.63" x2="-29.21" y2="74.93" width="0" layer="19" extent="1-1"/>
 <wire x1="-19.685" y1="91.9734" x2="-29.08" y2="87.63" width="0" layer="19" extent="1-1"/>
@@
 <contactref element="U$2" pad="3.3V2"/>
 <contactref element="R1" pad="1"/>
-<contactref element="U$1" pad="VOUT"/>
 <contactref element="C2" pad="+"/>
 <contactref element="C3" pad="1"/>
@@
 <contactref element="IC4" pad="10"/>
 <contactref element="IC3" pad="10"/>
-<wire x1="-175.895" y1="-263.6266" x2="-183.515" y2="-263.6266" width="0" layer="19" extent="1-1"/>
+<contactref element="U$6" pad="VOUT"/>
+<wire x1="-175.895" y1="-263.6266" x2="-167.64" y2="-290.83" width="0" layer="19" extent="1-1"/>
+<wire x1="-183.515" y1="-263.6266" x2="-175.895" y2="-263.6266" width="0" layer="19" extent="1-1"/>
 <wire x1="-146.685" y1="-263.6266" x2="-175.895" y2="-263.6266" width="0" layer="19" extent="1-1"/>
 <wire x1="-139.065" y1="-263.6266" x2="-146.685" y2="-263.6266" width="0" layer="19" extent="1-1"/>
@@
 <wire x1="-30.48" y1="30.48" x2="-35.56" y2="17.78" width="0" layer="19" extent="1-1"/>
 <wire x1="-15.24" y1="55.88" x2="-30.48" y2="30.48" width="0" layer="19" extent="1-1"/>
-<wire x1="-15.24" y1="72.39" x2="-15.24" y2="55.88" width="0" layer="19" extent="1-1"/>
-<wire x1="-15.875" y1="91.9734" x2="-15.24" y2="72.39" width="0" layer="19" extent="1-1"/>
-<wire x1="-23.495" y1="91.9734" x2="-15.875" y2="91.9734" width="0" layer="19" extent="1-1"/>
-<wire x1="-31.88" y1="87.63" x2="-23.495" y2="91.9734" width="0" layer="19" extent="1-1"/>
+<wire x1="-31.88" y1="87.63" x2="-15.24" y2="55.88" width="0" layer="19" extent="1-1"/>
 <wire x1="-36.96" y1="87.63" x2="-31.88" y2="87.63" width="0" layer="19" extent="1-1"/>
+<wire x1="-23.495" y1="91.9734" x2="-31.88" y2="87.63" width="0" layer="19" extent="1-1"/>
+<wire x1="-15.875" y1="91.9734" x2="-23.495" y2="91.9734" width="0" layer="19" extent="1-1"/>
 <wire x1="-45.72" y1="74.93" x2="-36.96" y2="87.63" width="0" layer="19" extent="1-1"/>
 </signal>
@@
 <signal name="N$1">
 <contactref element="D1" pad="C"/>
-<contactref element="U$1" pad="VIN"/>
 <contactref element="C1" pad="+"/>
-<contactref element="U$1" pad="SHDN"/>
-<wire x1="-22.86" y1="72.39" x2="-20.32" y2="72.39" width="0" layer="19" extent="1-1"/>
-<wire x1="-34.29" y1="74.93" x2="-22.86" y2="72.39" width="0" layer="19" extent="1-1"/>
+<contactref element="U$6" pad="VIN"/>
+<wire x1="-34.29" y1="74.93" x2="-172.72" y2="-290.83" width="0" layer="19" extent="1-1"/>
 <wire x1="-49.19" y1="86.36" x2="-34.29" y2="74.93" width="0" layer="19" extent="1-1"/>
 </signal>

Commit message: base
Parts:
- added D10, D11, D12, D5, D6, D7, D8, D9: WHITE, SparkFun-LED:LED-1206
Changed lines of the file:
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@@
 <?xml version="1.0" encoding="utf-8"?>
 <!DOCTYPE eagle SYSTEM "eagle.dtd">
-<eagle version="8.5.0">
+<eagle version="8.6.2">
 <drawing>
 <settings>
@@
 <element name="IC4" library="74xx-us" library_urn="urn:adsk.eagle:library:88" package="SO16" package3d_urn="urn:adsk.eagle:package:2918/1" value="74LS595D" x="-179.07" y="-266.7"/>
 <element name="U$6" library="libreria valerio" package="REGOLATORE-3.3V-1A" value="REGOLATORE-3.3V-1A" x="-179.07" y="-292.1"/>
+<element name="D5" library="SparkFun-LED" package="LED-1206" value="WHITE" x="-184.15" y="-306.07">
+<attribute name="PROD_ID" value="DIO-09955" x="-184.15" y="-306.07" size="1.778" layer="27" display="off"/>
+</element>
+<element name="D6" library="SparkFun-LED" package="LED-1206" value="WHITE" x="-184.15" y="-311.15">
+<attribute name="PROD_ID" value="DIO-09955" x="-184.15" y="-311.15" size="1.778" layer="27" display="off"/>
+</element>
+<element name="D7" library="SparkFun-LED" package="LED-1206" value="WHITE" x="-184.15" y="-316.23">
+<attribute name="PROD_ID" value="DIO-09955" x="-184.15" y="-316.23" size="1.778" layer="27" display="off"/>
+</element>
+<element name="D8" library="SparkFun-LED" package="LED-1206" value="WHITE" x="-184.15" y="-321.31">
+<attribute name="PROD_ID" value="DIO-09955" x="-184.15" y="-321.31" size="1.778" layer="27" display="off"/>
+</element>
+<element name="D9" library="SparkFun-LED" package="LED-1206" value="WHITE" x="-184.15" y="-326.39">
+<attribute name="PROD_ID" value="DIO-09955" x="-184.15" y="-326.39" size="1.778" layer="27" display="off"/>
+</element>
+<element name="D10" library="SparkFun-LED" package="LED-1206" value="WHITE" x="-184.15" y="-331.47">
+<attribute name="PROD_ID" value="DIO-09955" x="-184.15" y="-331.47" size="1.778" layer="27" display="off"/>
+</element>
+<element name="D11" library="SparkFun-LED" package="LED-1206" value="WHITE" x="-184.15" y="-336.55">
+<attribute name="PROD_ID" value="DIO-09955" x="-184.15" y="-336.55" size="1.778" layer="27" display="off"/>
+</element>
+<element name="D12" library="SparkFun-LED" package="LED-1206" value="WHITE" x="-184.15" y="-341.63">
+<attribute name="PROD_ID" value="DIO-09955" x="-184.15" y="-341.63" size="1.778" layer="27" display="off"/>
+</element>
 </elements>
 <signals>

Commit message: base
Parts:
- added R10, R3, R4, R5, R6, R7, R8, R9: 180, rcl:0204/7
Connections:
- new net DIODO-1: D5.A, IC3.15
- new net DIODO-2: D6.A, IC3.1
- new net DIODO-3: D7.A, IC3.2
- new net DIODO-4: D8.A, IC3.3
- new net DIODO-5: D9.A, IC3.4
- new net DIODO-6: D10.A, IC3.5
- new net DIODO-7: D11.A, IC3.6
- new net DIODO-8: D12.A, IC3.7
- new net N$11: D8.C, R5.2
- new net N$12: D9.C, R7.2
- new net N$13: D10.C, R8.2
- new net N$14: D11.C, R9.2
- new net N$15: D12.C, R10.2
- new net N$7: D5.C, R3.2
- new net N$8: D6.C, R6.2
- new net N$9: D7.C, R4.2
Changed lines of the file:
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@@
 <attribute name="PROD_ID" value="DIO-09955" x="-184.15" y="-341.63" size="1.778" layer="27" display="off"/>
 </element>
+<element name="R6" library="rcl" library_urn="urn:adsk.eagle:library:334" package="0204/7" package3d_urn="urn:adsk.eagle:package:23498/1" value="180" x="-175.26" y="-351.79"/>
+<element name="R3" library="rcl" library_urn="urn:adsk.eagle:library:334" package="0204/7" package3d_urn="urn:adsk.eagle:package:23498/1" value="180" x="-175.26" y="-365.76"/>
+<element name="R4" library="rcl" library_urn="urn:adsk.eagle:library:334" package="0204/7" package3d_urn="urn:adsk.eagle:package:23498/1" value="180" x="-175.26" y="-379.73"/>
+<element name="R5" library="rcl" library_urn="urn:adsk.eagle:library:334" package="0204/7" package3d_urn="urn:adsk.eagle:package:23498/1" value="180" x="-175.26" y="-393.7"/>
+<element name="R7" library="rcl" library_urn="urn:adsk.eagle:library:334" package="0204/7" package3d_urn="urn:adsk.eagle:package:23498/1" value="180" x="-175.26" y="-407.67"/>
+<element name="R8" library="rcl" library_urn="urn:adsk.eagle:library:334" package="0204/7" package3d_urn="urn:adsk.eagle:package:23498/1" value="180" x="-175.26" y="-421.64"/>
+<element name="R9" library="rcl" library_urn="urn:adsk.eagle:library:334" package="0204/7" package3d_urn="urn:adsk.eagle:package:23498/1" value="180" x="-175.26" y="-435.61"/>
+<element name="R10" library="rcl" library_urn="urn:adsk.eagle:library:334" package="0204/7" package3d_urn="urn:adsk.eagle:package:23498/1" value="180" x="-175.26" y="-449.58"/>
 </elements>
 <signals>
@@
 <contactref element="IC4" pad="14"/>
 </signal>
+<signal name="DIODO-1">
+<contactref element="IC3" pad="15"/>
+<contactref element="D5" pad="A"/>
+<wire x1="-145.415" y1="-263.6266" x2="-185.65" y2="-306.07" width="0" layer="19" extent="1-1"/>
+</signal>
+<signal name="DIODO-2">
+<contactref element="IC3" pad="1"/>
+<contactref element="D6" pad="A"/>
+<wire x1="-146.685" y1="-269.7734" x2="-185.65" y2="-311.15" width="0" layer="19" extent="1-1"/>
+</signal>
+<signal name="DIODO-3">
+<contactref element="IC3" pad="2"/>
+<contactref element="D7" pad="A"/>
+<wire x1="-145.415" y1="-269.7734" x2="-185.65" y2="-316.23" width="0" layer="19" extent="1-1"/>
+</signal>
+<signal name="DIODO-4">
+<contactref element="IC3" pad="3"/>
+<contactref element="D8" pad="A"/>
+<wire x1="-144.145" y1="-269.7734" x2="-185.65" y2="-321.31" width="0" layer="19" extent="1-1"/>
+</signal>
+<signal name="DIODO-5">
+<contactref element="IC3" pad="4"/>
+<contactref element="D9" pad="A"/>
+<wire x1="-185.65" y1="-326.39" x2="-142.875" y2="-269.7734" width="0" layer="19" extent="1-1"/>
+</signal>
+<signal name="DIODO-6">
+<contactref element="IC3" pad="5"/>
+<contactref element="D10" pad="A"/>
+<wire x1="-185.65" y1="-331.47" x2="-141.605" y2="-269.7734" width="0" layer="19" extent="1-1"/>
+</signal>
+<signal name="DIODO-7">
+<contactref element="IC3" pad="6"/>
+<contactref element="D11" pad="A"/>
+<wire x1="-185.65" y1="-336.55" x2="-140.335" y2="-269.7734" width="0" layer="19" extent="1-1"/>
+</signal>
+<signal name="DIODO-8">
+<contactref element="IC3" pad="7"/>
+<contactref element="D12" pad="A"/>
+<wire x1="-185.65" y1="-341.63" x2="-139.065" y2="-269.7734" width="0" layer="19" extent="1-1"/>
+</signal>
+<signal name="N$7">
+<contactref element="D5" pad="C"/>
+<contactref element="R3" pad="2"/>
+<wire x1="-171.45" y1="-365.76" x2="-182.65" y2="-306.07" width="0" layer="19" extent="1-1"/>
+</signal>
+<signal name="N$8">
+<contactref element="D6" pad="C"/>
+<contactref element="R6" pad="2"/>
+<wire x1="-171.45" y1="-351.79" x2="-182.65" y2="-311.15" width="0" layer="19" extent="1-1"/>
+</signal>
+<signal name="N$9">
+<contactref element="D7" pad="C"/>
+<contactref element="R4" pad="2"/>
+<wire x1="-171.45" y1="-379.73" x2="-182.65" y2="-316.23" width="0" layer="19" extent="1-1"/>
+</signal>
+<signal name="N$11">
+<contactref element="D8" pad="C"/>
+<contactref element="R5" pad="2"/>
+<wire x1="-171.45" y1="-393.7" x2="-182.65" y2="-321.31" width="0" layer="19" extent="1-1"/>
+</signal>
+<signal name="N$12">
+<contactref element="D9" pad="C"/>
+<contactref element="R7" pad="2"/>
+<wire x1="-171.45" y1="-407.67" x2="-182.65" y2="-326.39" width="0" layer="19" extent="1-1"/>
+</signal>
+<signal name="N$13">
+<contactref element="D10" pad="C"/>
+<contactref element="R8" pad="2"/>
+<wire x1="-182.65" y1="-331.47" x2="-171.45" y2="-421.64" width="0" layer="19" extent="1-1"/>
+</signal>
+<signal name="N$14">
+<contactref element="D11" pad="C"/>
+<contactref element="R9" pad="2"/>
+<wire x1="-182.65" y1="-336.55" x2="-171.45" y2="-435.61" width="0" layer="19" extent="1-1"/>
+</signal>
+<signal name="N$15">
+<contactref element="D12" pad="C"/>
+<contactref element="R10" pad="2"/>
+<wire x1="-182.65" y1="-341.63" x2="-171.45" y2="-449.58" width="0" layer="19" extent="1-1"/>
+</signal>
 </signals>

Commit message: base
Connections:
- removed net N$5: IC3.14
- new net SR1: IC2.9, IC3.14
- net GND: now also R10.1, R3.1, R4.1, R5.1, R6.1, R7.1, R8.1, R9.1, U$6.GND
Changed lines of the file:
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@@
 <contactref element="IC3" pad="13"/>
 <contactref element="IC4" pad="13"/>
+<contactref element="U$6" pad="GND"/>
+<contactref element="R10" pad="1"/>
+<contactref element="R9" pad="1"/>
+<contactref element="R8" pad="1"/>
+<contactref element="R7" pad="1"/>
+<contactref element="R5" pad="1"/>
+<contactref element="R4" pad="1"/>
+<contactref element="R6" pad="1"/>
+<contactref element="R3" pad="1"/>
 <wire x1="-30.48" y1="-165.1" x2="-64.77" y2="-171.45" width="0" layer="19" extent="1-1"/>
 <wire x1="-30.48" y1="-160.02" x2="-30.48" y2="-165.1" width="0" layer="19" extent="1-1"/>
@@
 <wire x1="-174.625" y1="-269.7734" x2="-142.875" y2="-263.6266" width="0" layer="19" extent="1-1"/>
 <wire x1="-179.705" y1="-263.6266" x2="-174.625" y2="-269.7734" width="0" layer="19" extent="1-1"/>
+<wire x1="-170.18" y1="-290.83" x2="-174.625" y2="-269.7734" width="0" layer="19" extent="1-1"/>
+<wire x1="-179.07" y1="-351.79" x2="-170.18" y2="-290.83" width="0" layer="19" extent="1-1"/>
+<wire x1="-179.07" y1="-365.76" x2="-179.07" y2="-351.79" width="0" layer="19" extent="1-1"/>
+<wire x1="-179.07" y1="-379.73" x2="-179.07" y2="-365.76" width="0" layer="19" extent="1-1"/>
+<wire x1="-179.07" y1="-393.7" x2="-179.07" y2="-379.73" width="0" layer="19" extent="1-1"/>
+<wire x1="-179.07" y1="-407.67" x2="-179.07" y2="-393.7" width="0" layer="19" extent="1-1"/>
+<wire x1="-179.07" y1="-421.64" x2="-179.07" y2="-407.67" width="0" layer="19" extent="1-1"/>
+<wire x1="-179.07" y1="-435.61" x2="-179.07" y2="-421.64" width="0" layer="19" extent="1-1"/>
+<wire x1="-179.07" y1="-449.58" x2="-179.07" y2="-435.61" width="0" layer="19" extent="1-1"/>
 </signal>
 <signal name="VIN">
@@
 <wire x1="-62.19" y1="-226.06" x2="-64.77" y2="-80.01" width="0" layer="19" extent="1-1"/>
 </signal>
-<signal name="N$5">
-<contactref element="IC3" pad="14"/>
-</signal>
 <signal name="N$10">
 <contactref element="IC4" pad="14"/>
@@
 <wire x1="-182.65" y1="-341.63" x2="-171.45" y2="-449.58" width="0" layer="19" extent="1-1"/>
 </signal>
+<signal name="SR1">
+<contactref element="IC2" pad="9"/>
+<contactref element="IC3" pad="14"/>
+<wire x1="-14.605" y1="91.9734" x2="-144.145" y2="-263.6266" width="0" layer="19" extent="1-1"/>
+</signal>
 </signals>
