File: hardware/electronics/Base/base.brd (EAGLE design)
At the start: 160 x 100 mm, 41 parts, among them IC1 7805T, IC2 74LS595D, IC3 74LS595D, IC4 74LS595D

Commit message: base+
Parts:
- added SV1, SV2, SV3, SV4: (no value), con-lstb:MA03-2
Connections:
- new net ALERT-1: SV1.5
- new net ALERT-2: SV3.5
- new net ALERT-3: SV2.5
- new net ALERT-4: SV4.5
- new net N$22: SV3.3
- new net N$25: SV1.3
- new net N$34: SV4.3
- new net N$37: SV2.3
- new net SCL: SV1.2, SV2.2, SV3.2, SV4.2
- new net SDA: SV1.4, SV2.4, SV3.4, SV4.4
- net 3.3V: now also SV1.6, SV2.6, SV3.6, SV4.6
- net GND: now also SV1.1, SV2.1, SV3.1, SV4.1
Changed lines of the file:
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@@
 <?xml version="1.0" encoding="utf-8"?>
 <!DOCTYPE eagle SYSTEM "eagle.dtd">
-<eagle version="8.6.2">
+<eagle version="8.6.3">
 <drawing>
 <settings>
@@
 <element name="R9" library="rcl" library_urn="urn:adsk.eagle:library:334" package="0204/7" package3d_urn="urn:adsk.eagle:package:23498/1" value="180" x="-175.26" y="-435.61"/>
 <element name="R10" library="rcl" library_urn="urn:adsk.eagle:library:334" package="0204/7" package3d_urn="urn:adsk.eagle:package:23498/1" value="180" x="-175.26" y="-449.58"/>
+<element name="SV1" library="con-lstb" library_urn="urn:adsk.eagle:library:162" package="MA03-2" package3d_urn="urn:adsk.eagle:package:8334/1" value="" x="-175.26" y="-466.09">
+<attribute name="MF" value="" x="-175.26" y="-466.09" size="1.778" layer="27" display="off"/>
+<attribute name="MPN" value="" x="-175.26" y="-466.09" size="1.778" layer="27" display="off"/>
+<attribute name="OC_FARNELL" value="unknown" x="-175.26" y="-466.09" size="1.778" layer="27" display="off"/>
+<attribute name="OC_NEWARK" value="unknown" x="-175.26" y="-466.09" size="1.778" layer="27" display="off"/>
+</element>
+<element name="SV2" library="con-lstb" library_urn="urn:adsk.eagle:library:162" package="MA03-2" package3d_urn="urn:adsk.eagle:package:8334/1" value="" x="-175.26" y="-483.87">
+<attribute name="MF" value="" x="-175.26" y="-483.87" size="1.778" layer="27" display="off"/>
+<attribute name="MPN" value="" x="-175.26" y="-483.87" size="1.778" layer="27" display="off"/>
+<attribute name="OC_FARNELL" value="unknown" x="-175.26" y="-483.87" size="1.778" layer="27" display="off"/>
+<attribute name="OC_NEWARK" value="unknown" x="-175.26" y="-483.87" size="1.778" layer="27" display="off"/>
+</element>
+<element name="SV3" library="con-lstb" library_urn="urn:adsk.eagle:library:162" package="MA03-2" package3d_urn="urn:adsk.eagle:package:8334/1" value="" x="-175.26" y="-501.65">
+<attribute name="MF" value="" x="-175.26" y="-501.65" size="1.778" layer="27" display="off"/>
+<attribute name="MPN" value="" x="-175.26" y="-501.65" size="1.778" layer="27" display="off"/>
+<attribute name="OC_FARNELL" value="unknown" x="-175.26" y="-501.65" size="1.778" layer="27" display="off"/>
+<attribute name="OC_NEWARK" value="unknown" x="-175.26" y="-501.65" size="1.778" layer="27" display="off"/>
+</element>
+<element name="SV4" library="con-lstb" library_urn="urn:adsk.eagle:library:162" package="MA03-2" package3d_urn="urn:adsk.eagle:package:8334/1" value="" x="-175.26" y="-519.43">
+<attribute name="MF" value="" x="-175.26" y="-519.43" size="1.778" layer="27" display="off"/>
+<attribute name="MPN" value="" x="-175.26" y="-519.43" size="1.778" layer="27" display="off"/>
+<attribute name="OC_FARNELL" value="unknown" x="-175.26" y="-519.43" size="1.778" layer="27" display="off"/>
+<attribute name="OC_NEWARK" value="unknown" x="-175.26" y="-519.43" size="1.778" layer="27" display="off"/>
+</element>
 </elements>
 <signals>
@@
 <contactref element="R6" pad="1"/>
 <contactref element="R3" pad="1"/>
+<contactref element="SV1" pad="1"/>
+<contactref element="SV3" pad="1"/>
+<contactref element="SV4" pad="1"/>
+<contactref element="SV2" pad="1"/>
 <wire x1="-30.48" y1="-165.1" x2="-64.77" y2="-171.45" width="0" layer="19" extent="1-1"/>
 <wire x1="-30.48" y1="-160.02" x2="-30.48" y2="-165.1" width="0" layer="19" extent="1-1"/>
@@
 <wire x1="-179.07" y1="-435.61" x2="-179.07" y2="-421.64" width="0" layer="19" extent="1-1"/>
 <wire x1="-179.07" y1="-449.58" x2="-179.07" y2="-435.61" width="0" layer="19" extent="1-1"/>
+<wire x1="-177.8" y1="-467.36" x2="-179.07" y2="-449.58" width="0" layer="19" extent="1-1"/>
+<wire x1="-177.8" y1="-485.14" x2="-177.8" y2="-467.36" width="0" layer="19" extent="1-1"/>
+<wire x1="-177.8" y1="-502.92" x2="-177.8" y2="-485.14" width="0" layer="19" extent="1-1"/>
+<wire x1="-177.8" y1="-520.7" x2="-177.8" y2="-502.92" width="0" layer="19" extent="1-1"/>
 </signal>
 <signal name="VIN">
@@
 <contactref element="IC3" pad="10"/>
 <contactref element="U$6" pad="VOUT"/>
+<contactref element="SV1" pad="6"/>
+<contactref element="SV3" pad="6"/>
+<contactref element="SV2" pad="6"/>
+<contactref element="SV4" pad="6"/>
 <wire x1="-175.895" y1="-263.6266" x2="-167.64" y2="-290.83" width="0" layer="19" extent="1-1"/>
 <wire x1="-183.515" y1="-263.6266" x2="-175.895" y2="-263.6266" width="0" layer="19" extent="1-1"/>
 <wire x1="-146.685" y1="-263.6266" x2="-175.895" y2="-263.6266" width="0" layer="19" extent="1-1"/>
 <wire x1="-139.065" y1="-263.6266" x2="-146.685" y2="-263.6266" width="0" layer="19" extent="1-1"/>
+<wire x1="-172.72" y1="-464.82" x2="-167.64" y2="-290.83" width="0" layer="19" extent="1-1"/>
+<wire x1="-172.72" y1="-482.6" x2="-172.72" y2="-464.82" width="0" layer="19" extent="1-1"/>
+<wire x1="-172.72" y1="-500.38" x2="-172.72" y2="-482.6" width="0" layer="19" extent="1-1"/>
+<wire x1="-172.72" y1="-518.16" x2="-172.72" y2="-500.38" width="0" layer="19" extent="1-1"/>
 <wire x1="-40.64" y1="2.54" x2="-139.065" y2="-263.6266" width="0" layer="19" extent="1-1"/>
 <wire x1="-35.56" y1="17.78" x2="-40.64" y2="2.54" width="0" layer="19" extent="1-1"/>
@@
 <wire x1="-14.605" y1="91.9734" x2="-144.145" y2="-263.6266" width="0" layer="19" extent="1-1"/>
 </signal>
+<signal name="SDA">
+<contactref element="SV1" pad="4"/>
+<contactref element="SV3" pad="4"/>
+<contactref element="SV2" pad="4"/>
+<contactref element="SV4" pad="4"/>
+<wire x1="-175.26" y1="-500.38" x2="-175.26" y2="-518.16" width="0" layer="19" extent="1-1"/>
+<wire x1="-175.26" y1="-482.6" x2="-175.26" y2="-500.38" width="0" layer="19" extent="1-1"/>
+<wire x1="-175.26" y1="-464.82" x2="-175.26" y2="-482.6" width="0" layer="19" extent="1-1"/>
+</signal>
+<signal name="SCL">
+<contactref element="SV1" pad="2"/>
+<contactref element="SV3" pad="2"/>
+<contactref element="SV4" pad="2"/>
+<contactref element="SV2" pad="2"/>
+<wire x1="-177.8" y1="-500.38" x2="-177.8" y2="-518.16" width="0" layer="19" extent="1-1"/>
+<wire x1="-177.8" y1="-482.6" x2="-177.8" y2="-500.38" width="0" layer="19" extent="1-1"/>
+<wire x1="-177.8" y1="-464.82" x2="-177.8" y2="-482.6" width="0" layer="19" extent="1-1"/>
+</signal>
+<signal name="N$22">
+<contactref element="SV3" pad="3"/>
+</signal>
+<signal name="ALERT-2">
+<contactref element="SV3" pad="5"/>
+</signal>
+<signal name="N$25">
+<contactref element="SV1" pad="3"/>
+</signal>
+<signal name="ALERT-1">
+<contactref element="SV1" pad="5"/>
+</signal>
+<signal name="N$34">
+<contactref element="SV4" pad="3"/>
+</signal>
+<signal name="ALERT-4">
+<contactref element="SV4" pad="5"/>
+</signal>
+<signal name="N$37">
+<contactref element="SV2" pad="3"/>
+</signal>
+<signal name="ALERT-3">
+<contactref element="SV2" pad="5"/>
+</signal>
 </signals>

Commit message: Base
Connections:
- net DIODO-1 renamed LED-1
- net DIODO-2 renamed LED-2
- net DIODO-3 renamed LED-3
- net DIODO-4 renamed LED-4
- net DIODO-5 renamed LED-5
- net DIODO-6 renamed LED-6
- net DIODO-7 renamed LED-7
- net DIODO-8 renamed LED-8
- removed net N$10: IC4.14
- new net SR2: IC3.9, IC4.14
Changed lines of the file:
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@@
 <wire x1="-62.19" y1="-226.06" x2="-64.77" y2="-80.01" width="0" layer="19" extent="1-1"/>
-</signal>
-<signal name="N$10">
-<contactref element="IC4" pad="14"/>
-</signal>
-<signal name="DIODO-1">
-<contactref element="IC3" pad="15"/>
-<contactref element="D5" pad="A"/>
-<wire x1="-145.415" y1="-263.6266" x2="-185.65" y2="-306.07" width="0" layer="19" extent="1-1"/>
-</signal>
-<signal name="DIODO-2">
-<contactref element="IC3" pad="1"/>
-<contactref element="D6" pad="A"/>
-<wire x1="-146.685" y1="-269.7734" x2="-185.65" y2="-311.15" width="0" layer="19" extent="1-1"/>
-</signal>
-<signal name="DIODO-3">
-<contactref element="IC3" pad="2"/>
-<contactref element="D7" pad="A"/>
-<wire x1="-145.415" y1="-269.7734" x2="-185.65" y2="-316.23" width="0" layer="19" extent="1-1"/>
-</signal>
-<signal name="DIODO-4">
-<contactref element="IC3" pad="3"/>
-<contactref element="D8" pad="A"/>
-<wire x1="-144.145" y1="-269.7734" x2="-185.65" y2="-321.31" width="0" layer="19" extent="1-1"/>
-</signal>
-<signal name="DIODO-5">
-<contactref element="IC3" pad="4"/>
-<contactref element="D9" pad="A"/>
-<wire x1="-185.65" y1="-326.39" x2="-142.875" y2="-269.7734" width="0" layer="19" extent="1-1"/>
-</signal>
-<signal name="DIODO-6">
-<contactref element="IC3" pad="5"/>
-<contactref element="D10" pad="A"/>
-<wire x1="-185.65" y1="-331.47" x2="-141.605" y2="-269.7734" width="0" layer="19" extent="1-1"/>
-</signal>
-<signal name="DIODO-7">
-<contactref element="IC3" pad="6"/>
-<contactref element="D11" pad="A"/>
-<wire x1="-185.65" y1="-336.55" x2="-140.335" y2="-269.7734" width="0" layer="19" extent="1-1"/>
-</signal>
-<signal name="DIODO-8">
-<contactref element="IC3" pad="7"/>
-<contactref element="D12" pad="A"/>
-<wire x1="-185.65" y1="-341.63" x2="-139.065" y2="-269.7734" width="0" layer="19" extent="1-1"/>
 </signal>
 <signal name="N$7">
@@
 <contactref element="SV2" pad="5"/>
 </signal>
+<signal name="LED-1">
+<contactref element="IC3" pad="15"/>
+<contactref element="D5" pad="A"/>
+<wire x1="-145.415" y1="-263.6266" x2="-185.65" y2="-306.07" width="0" layer="19" extent="1-1"/>
+</signal>
+<signal name="LED-2">
+<contactref element="IC3" pad="1"/>
+<contactref element="D6" pad="A"/>
+<wire x1="-146.685" y1="-269.7734" x2="-185.65" y2="-311.15" width="0" layer="19" extent="1-1"/>
+</signal>
+<signal name="LED-3">
+<contactref element="IC3" pad="2"/>
+<contactref element="D7" pad="A"/>
+<wire x1="-145.415" y1="-269.7734" x2="-185.65" y2="-316.23" width="0" layer="19" extent="1-1"/>
+</signal>
+<signal name="LED-4">
+<contactref element="IC3" pad="3"/>
+<contactref element="D8" pad="A"/>
+<wire x1="-144.145" y1="-269.7734" x2="-185.65" y2="-321.31" width="0" layer="19" extent="1-1"/>
+</signal>
+<signal name="LED-5">
+<contactref element="IC3" pad="4"/>
+<contactref element="D9" pad="A"/>
+<wire x1="-185.65" y1="-326.39" x2="-142.875" y2="-269.7734" width="0" layer="19" extent="1-1"/>
+</signal>
+<signal name="LED-6">
+<contactref element="IC3" pad="5"/>
+<contactref element="D10" pad="A"/>
+<wire x1="-185.65" y1="-331.47" x2="-141.605" y2="-269.7734" width="0" layer="19" extent="1-1"/>
+</signal>
+<signal name="LED-7">
+<contactref element="IC3" pad="6"/>
+<contactref element="D11" pad="A"/>
+<wire x1="-185.65" y1="-336.55" x2="-140.335" y2="-269.7734" width="0" layer="19" extent="1-1"/>
+</signal>
+<signal name="LED-8">
+<contactref element="IC3" pad="7"/>
+<contactref element="D12" pad="A"/>
+<wire x1="-185.65" y1="-341.63" x2="-139.065" y2="-269.7734" width="0" layer="19" extent="1-1"/>
+</signal>
+<signal name="SR2">
+<contactref element="IC3" pad="9"/>
+<contactref element="IC4" pad="14"/>
+<wire x1="-137.795" y1="-263.6266" x2="-180.975" y2="-263.6266" width="0" layer="19" extent="1-1"/>
+</signal>
 </signals>

Commit message: Collegate le linee alla basa
Connections:
- removed net N$22: SV3.3
- removed net N$25: SV1.3
- removed net N$34: SV4.3
- removed net N$37: SV2.3
- net 3.3V: now also SV2.3
- net GND: now also SV1.3
- net SCL: now also SV4.3, U$2.19/A5
- net SDA: now also SV3.3, U$2.18/A4
Changed lines of the file:
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@@
 <?xml version="1.0" encoding="utf-8"?>
 <!DOCTYPE eagle SYSTEM "eagle.dtd">
-<eagle version="8.6.3">
+<eagle version="8.6.0">
 <drawing>
 <settings>
@@
 <contactref element="SV4" pad="1"/>
 <contactref element="SV2" pad="1"/>
+<contactref element="SV1" pad="3"/>
 <wire x1="-30.48" y1="-165.1" x2="-64.77" y2="-171.45" width="0" layer="19" extent="1-1"/>
 <wire x1="-30.48" y1="-160.02" x2="-30.48" y2="-165.1" width="0" layer="19" extent="1-1"/>
@@
 <wire x1="-179.07" y1="-449.58" x2="-179.07" y2="-435.61" width="0" layer="19" extent="1-1"/>
 <wire x1="-177.8" y1="-467.36" x2="-179.07" y2="-449.58" width="0" layer="19" extent="1-1"/>
+<wire x1="-175.26" y1="-467.36" x2="-177.8" y2="-467.36" width="0" layer="19" extent="1-1"/>
 <wire x1="-177.8" y1="-485.14" x2="-177.8" y2="-467.36" width="0" layer="19" extent="1-1"/>
 <wire x1="-177.8" y1="-502.92" x2="-177.8" y2="-485.14" width="0" layer="19" extent="1-1"/>
@@
 <contactref element="SV2" pad="6"/>
 <contactref element="SV4" pad="6"/>
+<contactref element="SV2" pad="3"/>
 <wire x1="-175.895" y1="-263.6266" x2="-167.64" y2="-290.83" width="0" layer="19" extent="1-1"/>
 <wire x1="-183.515" y1="-263.6266" x2="-175.895" y2="-263.6266" width="0" layer="19" extent="1-1"/>
@@
 <wire x1="-172.72" y1="-464.82" x2="-167.64" y2="-290.83" width="0" layer="19" extent="1-1"/>
 <wire x1="-172.72" y1="-482.6" x2="-172.72" y2="-464.82" width="0" layer="19" extent="1-1"/>
-<wire x1="-172.72" y1="-500.38" x2="-172.72" y2="-482.6" width="0" layer="19" extent="1-1"/>
+<wire x1="-175.26" y1="-485.14" x2="-172.72" y2="-482.6" width="0" layer="19" extent="1-1"/>
+<wire x1="-172.72" y1="-500.38" x2="-175.26" y2="-485.14" width="0" layer="19" extent="1-1"/>
 <wire x1="-172.72" y1="-518.16" x2="-172.72" y2="-500.38" width="0" layer="19" extent="1-1"/>
 <wire x1="-40.64" y1="2.54" x2="-139.065" y2="-263.6266" width="0" layer="19" extent="1-1"/>
@@
 <contactref element="SV2" pad="4"/>
 <contactref element="SV4" pad="4"/>
-<wire x1="-175.26" y1="-500.38" x2="-175.26" y2="-518.16" width="0" layer="19" extent="1-1"/>
+<contactref element="SV3" pad="3"/>
+<contactref element="U$2" pad="18/A4"/>
+<wire x1="-175.26" y1="-502.92" x2="-175.26" y2="-518.16" width="0" layer="19" extent="1-1"/>
+<wire x1="-175.26" y1="-500.38" x2="-175.26" y2="-502.92" width="0" layer="19" extent="1-1"/>
 <wire x1="-175.26" y1="-482.6" x2="-175.26" y2="-500.38" width="0" layer="19" extent="1-1"/>
 <wire x1="-175.26" y1="-464.82" x2="-175.26" y2="-482.6" width="0" layer="19" extent="1-1"/>
+<wire x1="-30.48" y1="15.24" x2="-175.26" y2="-464.82" width="0" layer="19" extent="1-1"/>
 </signal>
 <signal name="SCL">
@@
 <contactref element="SV4" pad="2"/>
 <contactref element="SV2" pad="2"/>
+<contactref element="SV4" pad="3"/>
+<contactref element="U$2" pad="19/A5"/>
+<wire x1="-175.26" y1="-520.7" x2="-177.8" y2="-518.16" width="0" layer="19" extent="1-1"/>
 <wire x1="-177.8" y1="-500.38" x2="-177.8" y2="-518.16" width="0" layer="19" extent="1-1"/>
 <wire x1="-177.8" y1="-482.6" x2="-177.8" y2="-500.38" width="0" layer="19" extent="1-1"/>
 <wire x1="-177.8" y1="-464.82" x2="-177.8" y2="-482.6" width="0" layer="19" extent="1-1"/>
-</signal>
-<signal name="N$22">
-<contactref element="SV3" pad="3"/>
+<wire x1="-30.48" y1="17.78" x2="-177.8" y2="-464.82" width="0" layer="19" extent="1-1"/>
 </signal>
 <signal name="ALERT-2">
 <contactref element="SV3" pad="5"/>
 </signal>
-<signal name="N$25">
-<contactref element="SV1" pad="3"/>
-</signal>
 <signal name="ALERT-1">
 <contactref element="SV1" pad="5"/>
 </signal>
-<signal name="N$34">
-<contactref element="SV4" pad="3"/>
-</signal>
 <signal name="ALERT-4">
 <contactref element="SV4" pad="5"/>
 </signal>
-<signal name="N$37">
-<contactref element="SV2" pad="3"/>
-</signal>
 <signal name="ALERT-3">
