File: hardware/electronics/Base/base.sch (EAGLE design)
At the start: 15 parts, among them IC1 7805T, IC2 74LS595D

Commit message: base aggiornata
Parts:
- added U$3: VHN5019, VHN5019:VHN5019
Connections:
- new net GND2: U$3.GND, U$3.GND2
- new net GNDM: U$3.GNDM
- net 3.3V: now also U$3.VDD
Changed lines of the file:
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@@
 <part name="U$2" library="Teensy_3_and_LC_Series_Boards_v1.4" deviceset="TEENSY_3.1-3.2_ALL_PINS&amp;PADS" device=""/>
 <part name="IC2" library="74xx-us" library_urn="urn:adsk.eagle:library:88" deviceset="74*595" device="D" package3d_urn="urn:adsk.eagle:package:2918/1" technology="LS"/>
+<part name="U$3" library="VHN5019" deviceset="VHN5019" device=""/>
+<part name="GND3" library="supply1" library_urn="urn:adsk.eagle:library:371" deviceset="GND" device=""/>
+<part name="GND4" library="supply1" library_urn="urn:adsk.eagle:library:371" deviceset="GND" device=""/>
+<part name="SUPPLY4" library="SparkFun-PowerSymbols" deviceset="3.3V" device=""/>
 </parts>
 <sheets>
@@
 <instance part="U$2" gate="G$1" x="33.02" y="152.4"/>
 <instance part="IC2" gate="A" x="33.02" y="83.82"/>
+<instance part="U$3" gate="G$1" x="-55.88" y="86.36" rot="MR0"/>
+<instance part="GND3" gate="1" x="-43.18" y="99.06" rot="R90"/>
+<instance part="GND4" gate="1" x="-91.44" y="81.28" rot="R270"/>
+<instance part="SUPPLY4" gate="G$1" x="-48.26" y="91.44" rot="R270"/>
 </instances>
 <busses>
@@
 <junction x="-40.64" y="182.88"/>
 </segment>
+<segment>
+<pinref part="SUPPLY4" gate="G$1" pin="3.3V"/>
+<pinref part="U$3" gate="G$1" pin="VDD"/>
+<wire x1="-48.26" y1="91.44" x2="-53.34" y2="91.44" width="0.1524" layer="91"/>
+</segment>
 </net>
 <net name="N$2" class="0">
@@
 </segment>
 </net>
+<net name="GND2" class="0">
+<segment>
+<pinref part="U$3" gate="G$1" pin="GND2"/>
+<wire x1="-53.34" y1="93.98" x2="-50.8" y2="93.98" width="0.1524" layer="91"/>
+<pinref part="GND3" gate="1" pin="GND"/>
+<pinref part="U$3" gate="G$1" pin="GND"/>
+<wire x1="-45.72" y1="99.06" x2="-50.8" y2="99.06" width="0.1524" layer="91"/>
+<wire x1="-50.8" y1="99.06" x2="-53.34" y2="99.06" width="0.1524" layer="91"/>
+<wire x1="-50.8" y1="93.98" x2="-50.8" y2="99.06" width="0.1524" layer="91"/>
+<junction x="-50.8" y="99.06"/>
+</segment>
+</net>
+<net name="GNDM" class="0">
+<segment>
+<pinref part="U$3" gate="G$1" pin="GNDM"/>
+<pinref part="GND4" gate="1" pin="GND"/>
+<wire x1="-81.28" y1="81.28" x2="-88.9" y2="81.28" width="0.1524" layer="91"/>
+</segment>
+</net>

Commit message: BASE
Parts:
- added U$4, U$5, U$7: VHN5019, VHN5019:VHN5019
Connections:
- new net MOT1_INA: IC2A.QA, U$3.INA
- new net MOT1_INB: U$3.INB
- new net MOT1_PWM: U$2.5/PWM, U$3.PWM
- new net MOT2_INA: IC2A.QC, U$5.INA
- new net MOT2_INB: IC2A.QB, IC2A.QD, U$5.INB
- new net MOT2_PWM: U$2.6/PWM, U$5.PWM
- new net MOT3_INA: IC2A.QE, U$4.INA
- new net MOT3_INB: IC2A.QF, U$4.INB
- new net MOT3_PWM: U$2.25/T/PWM, U$4.PWM
- new net MOT4_INA: IC2A.QG, U$7.INA
- new net MOT4_INB: IC2A.QH, U$7.INB
- new net MOT4_PWM: U$2.32/T/PWM, U$7.PWM
- new net VDD: U$4.VDD, U$5.VDD, U$7.VDD
- new net VMOT: U$3.VMOT, U$4.VMOT, U$5.VMOT, U$7.VMOT
- net 3.3V: now also IC2A.SCL, IC2P.VCC
- net GND: now also IC2A.G, IC2P.GND, U$4.GND, U$4.GND2, U$4.GNDM, U$5.GND, U$5.GND2, U$5.GNDM, U$7.GND, U$7.GND2, U$7.GNDM
Other:
- moved on the sheet: IC2

Commit message: base
Parts:
- added X1, X2, X3, X4: (no value), con-wago-500:W237-102
Connections:
- net MOT1_INA renamed MOT1-INA
- net MOT1_INB renamed MOT1-INB
- net MOT2_INA renamed MOT2-INA
- net MOT2_INB renamed MOT2-INB
- net MOT3_INA renamed MOT3-INA
- net MOT3_INB renamed MOT3-INB
- net MOT4_INA renamed MOT4-INA
- net MOT4_INB renamed MOT4-INB
- new net CLOCK: IC2A.SCK, U$2.27/A16
- new net DATA-IN: IC2A.SER, U$2.28/A17
- new net LATCH: IC2A.RCK, U$2.26/A15
- new net MOT1-PWM: U$3.PWM
- new net MOT2-PWM: U$5.PWM
- new net MOT3-PWM: U$4.PWM
- new net MOT4-PWM: U$7.PWM
- net MOT1_PWM: no longer U$3.PWM
- net MOT2_PWM: no longer U$5.PWM
- net MOT3_PWM: no longer U$4.PWM
- net MOT4_PWM: no longer U$7.PWM
Other:
- moved on the sheet: IC2, IC2P

Commit message: base
Connections:
- new net MOTORE1-1: U$3.INMOT1, X1-1.KL
- new net MOTORE1-2: U$3.INMOT2, X1-2.KL
- new net MOTORE2-1: U$5.INMOT1, X2-1.KL
- new net MOTORE2-2: U$5.INMOT2, X2-2.KL
- new net MOTORE3-1: U$4.INMOT1, X3-1.KL
- new net MOTORE3-2: U$4.INMOT2, X3-2.KL
- new net MOTORE4-1: U$7.INMOT1, X4-1.KL
- new net MOTORE4-2: U$7.INMOT2, X4-2.KL
Other:
- moved on the sheet: IC2, IC2P, U$3, U$4, U$5, U$7

Commit message: Base aggiornata
Other:
- note added: "Motor driver VHN5019"
- note added: "Pin motori"
- note added: "Shift register"
- note added: "Teensy 3.2"
- moved on the sheet: IC2, IC2P, U$2, U$4, U$5, U$7, X1-1, X1-2, X2-1, X2-2, X3-1, X3-2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

Commit message: base
Parts:
- added B1: SD_MMC_CARDSD_PCB, SparkFun-Boards:SD_MMC_CARDSD_PCB
- added IC3: 74LS595D, 74xx-us:74LS595D
Other:
- note added: "Shift register motori"
- note removed: "Shift register"
Changed lines of the file:
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@@
 <part name="X3" library="con-wago-500" library_urn="urn:adsk.eagle:library:195" deviceset="W237-102" device="" package3d_urn="urn:adsk.eagle:package:10688/1"/>
 <part name="X4" library="con-wago-500" library_urn="urn:adsk.eagle:library:195" deviceset="W237-102" device="" package3d_urn="urn:adsk.eagle:package:10688/1"/>
+<part name="FRAME2" library="frames" library_urn="urn:adsk.eagle:library:229" deviceset="A4L-LOC" device=""/>
+<part name="IC3" library="74xx-us" library_urn="urn:adsk.eagle:library:88" deviceset="74*595" device="D" package3d_urn="urn:adsk.eagle:package:2918/1" technology="LS"/>
+<part name="B1" library="SparkFun-Boards" deviceset="SD_MMC_CARD" device="SD_PCB"/>
 </parts>
 <sheets>
@@
 <wire x1="55.88" y1="81.28" x2="55.88" y2="111.76" width="1.27" layer="96" style="longdash"/>
 <wire x1="55.88" y1="81.28" x2="116.84" y2="81.28" width="1.27" layer="96" style="longdash"/>
-<text x="81.28" y="124.46" size="2.54" layer="99">Shift register</text>
+<text x="81.28" y="124.46" size="2.54" layer="99">Shift register motori</text>
 <wire x1="55.88" y1="111.76" x2="55.88" y2="129.54" width="1.27" layer="96" style="longdash"/>
 <wire x1="55.88" y1="129.54" x2="116.84" y2="129.54" width="1.27" layer="96" style="longdash"/>
@@
 </nets>
 </sheet>
+<sheet>
+<plain>
+</plain>
+<instances>
+<instance part="FRAME2" gate="G$1" x="0" y="0"/>
+<instance part="IC3" gate="A" x="66.04" y="116.84"/>
+<instance part="B1" gate="G$1" x="121.92" y="116.84"/>
+</instances>
+<busses>
+</busses>
+<nets>
+</nets>
+</sheet>

Commit message: aggiornamenti base
Parts:
- removed B1: SD_MMC_CARDSD_PCB, SparkFun-Boards:SD_MMC_CARDSD_PCB
- added DIS1: HD-H103, display-hp:HD-H103
- added IC4: 74LS595D, 74xx-us:74LS595D
Connections:
- net DATA-IN renamed DATA-IN1
- new net N$10: IC4A.SER
- new net N$5: IC3A.SER
- net 3.3V: now also IC3A.SCL, IC3P.VCC, IC4A.SCL, IC4P.VCC
- net CLOCK: now also IC3A.SCK, IC4A.SCK
- net GND: now also IC3A.G, IC3P.GND, IC4A.G, IC4P.GND
- net LATCH: now also IC3A.RCK, IC4A.RCK
Changed lines of the file:
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@@
 <part name="FRAME2" library="frames" library_urn="urn:adsk.eagle:library:229" deviceset="A4L-LOC" device=""/>
 <part name="IC3" library="74xx-us" library_urn="urn:adsk.eagle:library:88" deviceset="74*595" device="D" package3d_urn="urn:adsk.eagle:package:2918/1" technology="LS"/>
-<part name="B1" library="SparkFun-Boards" deviceset="SD_MMC_CARD" device="SD_PCB"/>
+<part name="GND13" library="supply1" library_urn="urn:adsk.eagle:library:371" deviceset="GND" device=""/>
+<part name="SUPPLY9" library="SparkFun-PowerSymbols" deviceset="3.3V" device=""/>
+<part name="DIS1" library="display-hp" library_urn="urn:adsk.eagle:library:212" deviceset="HD-H103" device="" package3d_urn="urn:adsk.eagle:package:13006/1"/>
+<part name="IC4" library="74xx-us" library_urn="urn:adsk.eagle:library:88" deviceset="74*595" device="D" package3d_urn="urn:adsk.eagle:package:2918/1" technology="LS"/>
+<part name="SUPPLY10" library="SparkFun-PowerSymbols" deviceset="3.3V" device=""/>
+<part name="GND14" library="supply1" library_urn="urn:adsk.eagle:library:371" deviceset="GND" device=""/>
+<part name="GND15" library="supply1" library_urn="urn:adsk.eagle:library:371" deviceset="GND" device=""/>
+<part name="GND16" library="supply1" library_urn="urn:adsk.eagle:library:371" deviceset="GND" device=""/>
+<part name="SUPPLY11" library="SparkFun-PowerSymbols" deviceset="3.3V" device=""/>
+<part name="SUPPLY12" library="SparkFun-PowerSymbols" deviceset="3.3V" device=""/>
 </parts>
 <sheets>
@@
 <wire x1="55.88" y1="81.28" x2="55.88" y2="111.76" width="1.27" layer="96" style="longdash"/>
 <wire x1="55.88" y1="81.28" x2="116.84" y2="81.28" width="1.27" layer="96" style="longdash"/>
-<text x="81.28" y="124.46" size="2.54" layer="99">Shift register motori</text>
+<text x="71.12" y="124.46" size="2.54" layer="99">Shift register motori</text>
 <wire x1="55.88" y1="111.76" x2="55.88" y2="129.54" width="1.27" layer="96" style="longdash"/>
 <wire x1="55.88" y1="129.54" x2="116.84" y2="129.54" width="1.27" layer="96" style="longdash"/>
@@
 <pinref part="IC2" gate="A" pin="RCK"/>
 <wire x1="78.74" y1="99.06" x2="76.2" y2="99.06" width="0.1524" layer="91"/>
-<label x="76.2" y="99.06" size="1.778" layer="95" rot="R180" xref="yes"/>
+<label x="76.2" y="99.06" size="1.27" layer="95" rot="R180" xref="yes"/>
 </segment>
 <segment>
@@
 <pinref part="IC2" gate="A" pin="SCK"/>
 <wire x1="78.74" y1="106.68" x2="76.2" y2="106.68" width="0.1524" layer="91"/>
-<label x="76.2" y="106.68" size="1.778" layer="95" rot="R180" xref="yes"/>
+<label x="76.2" y="106.68" size="1.27" layer="95" rot="R180" xref="yes"/>
 </segment>
 <segment>
@@
 </segment>
 </net>
-<net name="DATA-IN" class="0">
+<net name="DATA-IN1" class="0">
 <segment>
 <pinref part="IC2" gate="A" pin="SER"/>
 <wire x1="78.74" y1="111.76" x2="76.2" y2="111.76" width="0.1524" layer="91"/>
-<label x="76.2" y="111.76" size="1.778" layer="95" rot="R180" xref="yes"/>
+<label x="76.2" y="111.76" size="1.27" layer="95" rot="R180" xref="yes"/>
 </segment>
 <segment>
@@
 <instance part="FRAME2" gate="G$1" x="0" y="0"/>
 <instance part="IC3" gate="A" x="66.04" y="116.84"/>
-<instance part="B1" gate="G$1" x="121.92" y="116.84"/>
+<instance part="GND13" gate="1" x="53.34" y="134.62" rot="R270"/>
+<instance part="SUPPLY9" gate="G$1" x="76.2" y="134.62" rot="R270"/>
+<instance part="DIS1" gate="N" x="132.08" y="109.22"/>
+<instance part="IC4" gate="A" x="66.04" y="71.12"/>
+<instance part="IC3" gate="P" x="66.04" y="134.62" rot="R270"/>
+<instance part="IC4" gate="P" x="66.04" y="88.9" rot="R270"/>
+<instance part="SUPPLY10" gate="G$1" x="76.2" y="88.9" rot="R270"/>
+<instance part="GND14" gate="1" x="53.34" y="88.9" rot="R270"/>
+<instance part="GND15" gate="1" x="50.8" y="58.42" rot="R270"/>
+<instance part="GND16" gate="1" x="50.8" y="104.14" rot="R270"/>
+<instance part="SUPPLY11" gate="G$1" x="38.1" y="119.38" rot="R90"/>
+<instance part="SUPPLY12" gate="G$1" x="38.1" y="73.66" rot="R90"/>
 </instances>
 <busses>
 </busses>
 <nets>
+<net name="GND" class="0">
+<segment>
+<pinref part="GND13" gate="1" pin="GND"/>
+<pinref part="IC3" gate="P" pin="GND"/>
+</segment>
+<segment>
+<pinref part="GND14" gate="1" pin="GND"/>
+<pinref part="IC4" gate="P" pin="GND"/>
+</segment>
+<segment>
+<pinref part="IC3" gate="A" pin="G"/>
+<pinref part="GND16" gate="1" pin="GND"/>
+<wire x1="55.88" y1="104.14" x2="53.34" y2="104.14" width="0.1524" layer="91"/>
+</segment>
+<segment>
+<pinref part="IC4" gate="A" pin="G"/>
+<pinref part="GND15" gate="1" pin="GND"/>
+<wire x1="55.88" y1="58.42" x2="53.34" y2="58.42" width="0.1524" layer="91"/>
+</segment>
+</net>
+<net name="3.3V" class="0">
+<segment>
+<pinref part="IC3" gate="P" pin="VCC"/>
+<pinref part="SUPPLY9" gate="G$1" pin="3.3V"/>
+</segment>
+<segment>
+<pinref part="SUPPLY10" gate="G$1" pin="3.3V"/>
+<pinref part="IC4" gate="P" pin="VCC"/>
+</segment>
+<segment>
+<pinref part="IC4" gate="A" pin="SCL"/>
+<pinref part="SUPPLY12" gate="G$1" pin="3.3V"/>
+<wire x1="55.88" y1="73.66" x2="38.1" y2="73.66" width="0.1524" layer="91"/>
+</segment>
+<segment>
+<pinref part="IC3" gate="A" pin="SCL"/>
+<pinref part="SUPPLY11" gate="G$1" pin="3.3V"/>
+<wire x1="55.88" y1="119.38" x2="38.1" y2="119.38" width="0.1524" layer="91"/>
+</segment>
+</net>
+<net name="N$5" class="0">
+<segment>
+<pinref part="IC3" gate="A" pin="SER"/>
+<wire x1="55.88" y1="127" x2="50.8" y2="127" width="0.1524" layer="91"/>
+<label x="50.8" y="127" size="1.27" layer="95" rot="R180" xref="yes"/>
+</segment>
+</net>
+<net name="CLOCK" class="0">
+<segment>
+<pinref part="IC3" gate="A" pin="SCK"/>
+<wire x1="55.88" y1="121.92" x2="50.8" y2="121.92" width="0.1524" layer="91"/>
+<label x="50.8" y="121.92" size="1.27" layer="95" rot="R180" xref="yes"/>
+</segment>
+<segment>
+<pinref part="IC4" gate="A" pin="SCK"/>
+<wire x1="55.88" y1="76.2" x2="50.8" y2="76.2" width="0.1524" layer="91"/>
+<label x="50.8" y="76.2" size="1.27" layer="95" rot="R180" xref="yes"/>
+</segment>
+</net>
+<net name="LATCH" class="0">
+<segment>
+<pinref part="IC3" gate="A" pin="RCK"/>
+<wire x1="55.88" y1="114.3" x2="48.26" y2="114.3" width="0.1524" layer="91"/>
+<label x="48.26" y="114.3" size="1.27" layer="95" rot="R180" xref="yes"/>
+</segment>
+<segment>
+<pinref part="IC4" gate="A" pin="RCK"/>
+<wire x1="55.88" y1="68.58" x2="48.26" y2="68.58" width="0.1524" layer="91"/>
+<label x="48.26" y="68.58" size="1.27" layer="95" rot="R180" xref="yes"/>
+</segment>
+</net>
+<net name="N$10" class="0">
+<segment>
+<pinref part="IC4" gate="A" pin="SER"/>
+<wire x1="55.88" y1="81.28" x2="50.8" y2="81.28" width="0.1524" layer="91"/>
+<label x="50.8" y="81.28" size="1.27" layer="95" rot="R180" xref="yes"/>
+</segment>
+</net>
 </nets>
 </sheet>

Commit message: schema base piu lbr
Parts:
- removed DIS1: HD-H103, display-hp:HD-H103
- removed U$1: ALIM, Pololu switching alimentatore:ALIM
- added U$6: REGOLATORE-3.3V-1A, libreria valerio:REGOLATORE-3.3V-1A
Connections:
- net 3.3V: now also U$6.VOUT; no longer U$1.VOUT
- net GND: no longer U$1.GND
- net N$1: now also U$6.VIN; no longer U$1.SHDN, U$1.VIN
Changed lines of the file:
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@@
 </classes>
 <parts>
-<part name="U$1" library="Pololu switching alimentatore" deviceset="ALIM" device=""/>
 <part name="FRAME1" library="frames" library_urn="urn:adsk.eagle:library:229" deviceset="A4L-LOC" device=""/>
 <part name="C1" library="resistor" library_urn="urn:adsk.eagle:library:348" deviceset="CPOL-EU" device="E5-8.5" package3d_urn="urn:adsk.eagle:package:25860/1"/>
@@
 <part name="GND13" library="supply1" library_urn="urn:adsk.eagle:library:371" deviceset="GND" device=""/>
 <part name="SUPPLY9" library="SparkFun-PowerSymbols" deviceset="3.3V" device=""/>
-<part name="DIS1" library="display-hp" library_urn="urn:adsk.eagle:library:212" deviceset="HD-H103" device="" package3d_urn="urn:adsk.eagle:package:13006/1"/>
 <part name="IC4" library="74xx-us" library_urn="urn:adsk.eagle:library:88" deviceset="74*595" device="D" package3d_urn="urn:adsk.eagle:package:2918/1" technology="LS"/>
 <part name="SUPPLY10" library="SparkFun-PowerSymbols" deviceset="3.3V" device=""/>
@@
 <part name="SUPPLY11" library="SparkFun-PowerSymbols" deviceset="3.3V" device=""/>
 <part name="SUPPLY12" library="SparkFun-PowerSymbols" deviceset="3.3V" device=""/>
+<part name="U$6" library="libreria valerio" deviceset="REGOLATORE-3.3V-1A" device=""/>
 </parts>
 <sheets>
@@
 </plain>
 <instances>
-<instance part="U$1" gate="G$1" x="-63.5" y="182.88"/>
 <instance part="FRAME1" gate="G$1" x="-104.14" y="22.86"/>
 <instance part="C1" gate="G$1" x="-78.74" y="172.72"/>
@@
 <instance part="X4" gate="-1" x="63.5" y="58.42"/>
 <instance part="X4" gate="-2" x="63.5" y="53.34"/>
+<instance part="U$6" gate="G$1" x="-76.2" y="175.26"/>
 </instances>
 <busses>
@@
 <segment>
 <pinref part="D1" gate="G$1" pin="C"/>
-<pinref part="U$1" gate="G$1" pin="VIN"/>
 <wire x1="-83.82" y1="180.34" x2="-78.74" y2="180.34" width="0.1524" layer="91"/>
 <pinref part="C1" gate="G$1" pin="+"/>
-<wire x1="-78.74" y1="180.34" x2="-73.66" y2="180.34" width="0.1524" layer="91"/>
+<wire x1="-78.74" y1="180.34" x2="-76.2" y2="180.34" width="0.1524" layer="91"/>
+<wire x1="-76.2" y1="180.34" x2="-73.66" y2="180.34" width="0.1524" layer="91"/>
 <wire x1="-78.74" y1="175.26" x2="-78.74" y2="180.34" width="0.1524" layer="91"/>
 <junction x="-78.74" y="180.34"/>
-<pinref part="U$1" gate="G$1" pin="SHDN"/>
-<wire x1="-73.66" y1="185.42" x2="-78.74" y2="185.42" width="0.1524" layer="91"/>
-<wire x1="-78.74" y1="185.42" x2="-78.74" y2="180.34" width="0.1524" layer="91"/>
+<pinref part="U$6" gate="G$1" pin="VIN"/>
+<junction x="-76.2" y="180.34"/>
 </segment>
 </net>
@@
 <wire x1="-78.74" y1="167.64" x2="-78.74" y2="162.56" width="0.1524" layer="91"/>
 <wire x1="-78.74" y1="162.56" x2="-63.5" y2="162.56" width="0.1524" layer="91"/>
-<pinref part="U$1" gate="G$1" pin="GND"/>
-<wire x1="-63.5" y1="162.56" x2="-63.5" y2="175.26" width="0.1524" layer="91"/>
+<wire x1="-63.5" y1="162.56" x2="-63.5" y2="170.18" width="0.1524" layer="91"/>
 <junction x="-63.5" y="162.56"/>
 <pinref part="D2" gate="G$1" pin="C"/>
@@
 <pinref part="R1" gate="G$1" pin="1"/>
 <pinref part="SUPPLY1" gate="G$1" pin="3.3V"/>
-<pinref part="U$1" gate="G$1" pin="VOUT"/>
 <wire x1="-30.48" y1="182.88" x2="-40.64" y2="182.88" width="0.1524" layer="91"/>
 <junction x="-30.48" y="182.88"/>
@@
 <wire x1="-40.64" y1="177.8" x2="-40.64" y2="182.88" width="0.1524" layer="91"/>
 <junction x="-40.64" y="182.88"/>
+<pinref part="U$6" gate="G$1" pin="VOUT"/>
 </segment>
 <segment>
@@
 <instance part="GND13" gate="1" x="53.34" y="134.62" rot="R270"/>
 <instance part="SUPPLY9" gate="G$1" x="76.2" y="134.62" rot="R270"/>
-<instance part="DIS1" gate="N" x="132.08" y="109.22"/>
 <instance part="IC4" gate="A" x="66.04" y="71.12"/>
 <instance part="IC3" gate="P" x="66.04" y="134.62" rot="R270"/>
