File: hardware/electronics/Base/base.sch (EAGLE design)
At the start: 25 parts, among them IC1 7805T, IC2 74LS595D, IC3 74LS595D, IC4 74LS595D

Commit message: base
Parts:
- added D10, D11, D12, D5, D6, D7, D8, D9: WHITE, SparkFun-LED:LED-WHITE1206
Changed lines of the file:
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@@
 <?xml version="1.0" encoding="utf-8"?>
 <!DOCTYPE eagle SYSTEM "eagle.dtd">
-<eagle version="8.5.0">
+<eagle version="8.6.2">
 <drawing>
 <settings>
@@
 <part name="SUPPLY12" library="SparkFun-PowerSymbols" deviceset="3.3V" device=""/>
 <part name="U$6" library="libreria valerio" deviceset="REGOLATORE-3.3V-1A" device=""/>
+<part name="D5" library="SparkFun-LED" deviceset="LED-WHITE" device="1206" value="WHITE"/>
+<part name="D6" library="SparkFun-LED" deviceset="LED-WHITE" device="1206" value="WHITE"/>
+<part name="D7" library="SparkFun-LED" deviceset="LED-WHITE" device="1206" value="WHITE"/>
+<part name="D8" library="SparkFun-LED" deviceset="LED-WHITE" device="1206" value="WHITE"/>
+<part name="D9" library="SparkFun-LED" deviceset="LED-WHITE" device="1206" value="WHITE"/>
+<part name="D10" library="SparkFun-LED" deviceset="LED-WHITE" device="1206" value="WHITE"/>
+<part name="D11" library="SparkFun-LED" deviceset="LED-WHITE" device="1206" value="WHITE"/>
+<part name="D12" library="SparkFun-LED" deviceset="LED-WHITE" device="1206" value="WHITE"/>
 </parts>
 <sheets>
@@
 <instance part="SUPPLY11" gate="G$1" x="38.1" y="119.38" rot="R90"/>
 <instance part="SUPPLY12" gate="G$1" x="38.1" y="73.66" rot="R90"/>
+<instance part="D5" gate="G$1" x="101.6" y="127" rot="R90"/>
+<instance part="D6" gate="G$1" x="104.14" y="114.3" rot="R90"/>
+<instance part="D7" gate="G$1" x="104.14" y="104.14" rot="R90"/>
+<instance part="D8" gate="G$1" x="104.14" y="93.98" rot="R90"/>
+<instance part="D9" gate="G$1" x="106.68" y="83.82" rot="R90"/>
+<instance part="D10" gate="G$1" x="106.68" y="73.66" rot="R90"/>
+<instance part="D11" gate="G$1" x="109.22" y="63.5" rot="R90"/>
+<instance part="D12" gate="G$1" x="109.22" y="43.18" rot="R90"/>
 </instances>
 <busses>

Commit message: base
Parts:
- added R10, R3, R4, R5, R6, R7, R8, R9: 180, rcl:R-US_0204/7
Connections:
- new net DIODO-1: D5.A, IC3A.QA
- new net DIODO-2: D6.A, IC3A.QB
- new net DIODO-3: D7.A, IC3A.QC
- new net DIODO-4: D8.A, IC3A.QD
- new net DIODO-5: D9.A, IC3A.QE
- new net DIODO-6: D10.A, IC3A.QF
- new net DIODO-7: D11.A, IC3A.QG
- new net DIODO-8: D12.A, IC3A.QH
- new net N$11: D8.C, R5.2
- new net N$12: D9.C, R7.2
- new net N$13: D10.C, R8.2
- new net N$14: D11.C, R9.2
- new net N$15: D12.C, R10.2
- new net N$7: D5.C, R3.2
- new net N$8: D6.C, R6.2
- new net N$9: D7.C, R4.2
Other:
- moved on the sheet: D10, D11, D12, D5, D6, D7, D8, D9
Changed lines of the file:
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@@
 <part name="D11" library="SparkFun-LED" deviceset="LED-WHITE" device="1206" value="WHITE"/>
 <part name="D12" library="SparkFun-LED" deviceset="LED-WHITE" device="1206" value="WHITE"/>
+<part name="R6" library="rcl" library_urn="urn:adsk.eagle:library:334" deviceset="R-US_" device="0204/7" package3d_urn="urn:adsk.eagle:package:23498/1" value="180"/>
+<part name="R3" library="rcl" library_urn="urn:adsk.eagle:library:334" deviceset="R-US_" device="0204/7" package3d_urn="urn:adsk.eagle:package:23498/1" value="180"/>
+<part name="R4" library="rcl" library_urn="urn:adsk.eagle:library:334" deviceset="R-US_" device="0204/7" package3d_urn="urn:adsk.eagle:package:23498/1" value="180"/>
+<part name="R5" library="rcl" library_urn="urn:adsk.eagle:library:334" deviceset="R-US_" device="0204/7" package3d_urn="urn:adsk.eagle:package:23498/1" value="180"/>
+<part name="R7" library="rcl" library_urn="urn:adsk.eagle:library:334" deviceset="R-US_" device="0204/7" package3d_urn="urn:adsk.eagle:package:23498/1" value="180"/>
+<part name="R8" library="rcl" library_urn="urn:adsk.eagle:library:334" deviceset="R-US_" device="0204/7" package3d_urn="urn:adsk.eagle:package:23498/1" value="180"/>
+<part name="R9" library="rcl" library_urn="urn:adsk.eagle:library:334" deviceset="R-US_" device="0204/7" package3d_urn="urn:adsk.eagle:package:23498/1" value="180"/>
+<part name="R10" library="rcl" library_urn="urn:adsk.eagle:library:334" deviceset="R-US_" device="0204/7" package3d_urn="urn:adsk.eagle:package:23498/1" value="180"/>
 </parts>
 <sheets>
@@
 <instance part="SUPPLY11" gate="G$1" x="38.1" y="119.38" rot="R90"/>
 <instance part="SUPPLY12" gate="G$1" x="38.1" y="73.66" rot="R90"/>
-<instance part="D5" gate="G$1" x="101.6" y="127" rot="R90"/>
-<instance part="D6" gate="G$1" x="104.14" y="114.3" rot="R90"/>
-<instance part="D7" gate="G$1" x="104.14" y="104.14" rot="R90"/>
-<instance part="D8" gate="G$1" x="104.14" y="93.98" rot="R90"/>
-<instance part="D9" gate="G$1" x="106.68" y="83.82" rot="R90"/>
-<instance part="D10" gate="G$1" x="106.68" y="73.66" rot="R90"/>
-<instance part="D11" gate="G$1" x="109.22" y="63.5" rot="R90"/>
-<instance part="D12" gate="G$1" x="109.22" y="43.18" rot="R90"/>
+<instance part="D5" gate="G$1" x="119.38" y="127" rot="R90"/>
+<instance part="D6" gate="G$1" x="119.38" y="116.84" rot="R90"/>
+<instance part="D7" gate="G$1" x="119.38" y="106.68" rot="R90"/>
+<instance part="D8" gate="G$1" x="119.38" y="96.52" rot="R90"/>
+<instance part="D9" gate="G$1" x="119.38" y="86.36" rot="R90"/>
+<instance part="D10" gate="G$1" x="119.38" y="76.2" rot="R90"/>
+<instance part="D11" gate="G$1" x="119.38" y="66.04" rot="R90"/>
+<instance part="D12" gate="G$1" x="119.38" y="55.88" rot="R90"/>
+<instance part="R6" gate="G$1" x="132.08" y="116.84" rot="R180"/>
+<instance part="R3" gate="G$1" x="132.08" y="127" rot="R180"/>
+<instance part="R4" gate="G$1" x="132.08" y="106.68" rot="R180"/>
+<instance part="R5" gate="G$1" x="132.08" y="96.52" rot="R180"/>
+<instance part="R7" gate="G$1" x="132.08" y="86.36" rot="R180"/>
+<instance part="R8" gate="G$1" x="132.08" y="76.2" rot="R180"/>
+<instance part="R9" gate="G$1" x="132.08" y="66.04" rot="R180"/>
+<instance part="R10" gate="G$1" x="132.08" y="55.88" rot="R180"/>
 </instances>
 <busses>
@@
 </segment>
 </net>
+<net name="DIODO-1" class="0">
+<segment>
+<pinref part="IC3" gate="A" pin="QA"/>
+<wire x1="78.74" y1="127" x2="81.28" y2="127" width="0.1524" layer="91"/>
+<label x="81.28" y="127" size="1.27" layer="95" xref="yes"/>
+</segment>
+<segment>
+<pinref part="D5" gate="G$1" pin="A"/>
+<wire x1="116.84" y1="127" x2="114.3" y2="127" width="0.1524" layer="91"/>
+<label x="114.3" y="127" size="1.27" layer="95" rot="R180" xref="yes"/>
+</segment>
+</net>
+<net name="DIODO-2" class="0">
+<segment>
+<pinref part="IC3" gate="A" pin="QB"/>
+<wire x1="78.74" y1="124.46" x2="81.28" y2="124.46" width="0.1524" layer="91"/>
+<label x="81.28" y="124.46" size="1.27" layer="95" xref="yes"/>
+</segment>
+<segment>
+<pinref part="D6" gate="G$1" pin="A"/>
+<wire x1="116.84" y1="116.84" x2="114.3" y2="116.84" width="0.1524" layer="91"/>
+<label x="114.3" y="116.84" size="1.27" layer="95" rot="R180" xref="yes"/>
+</segment>
+</net>
+<net name="DIODO-3" class="0">
+<segment>
+<pinref part="IC3" gate="A" pin="QC"/>
+<wire x1="78.74" y1="121.92" x2="81.28" y2="121.92" width="0.1524" layer="91"/>
+<label x="81.28" y="121.92" size="1.27" layer="95" xref="yes"/>
+</segment>
+<segment>
+<pinref part="D7" gate="G$1" pin="A"/>
+<wire x1="116.84" y1="106.68" x2="114.3" y2="106.68" width="0.1524" layer="91"/>
+<label x="114.3" y="106.68" size="1.27" layer="95" rot="R180" xref="yes"/>
+</segment>
+</net>
+<net name="DIODO-4" class="0">
+<segment>
+<pinref part="IC3" gate="A" pin="QD"/>
+<wire x1="78.74" y1="119.38" x2="81.28" y2="119.38" width="0.1524" layer="91"/>
+<label x="81.28" y="119.38" size="1.27" layer="95" xref="yes"/>
+</segment>
+<segment>
+<pinref part="D8" gate="G$1" pin="A"/>
+<wire x1="116.84" y1="96.52" x2="114.3" y2="96.52" width="0.1524" layer="91"/>
+<label x="114.3" y="96.52" size="1.27" layer="95" rot="R180" xref="yes"/>
+</segment>
+</net>
+<net name="DIODO-5" class="0">
+<segment>
+<pinref part="IC3" gate="A" pin="QE"/>
+<wire x1="78.74" y1="116.84" x2="81.28" y2="116.84" width="0.1524" layer="91"/>
+<label x="81.28" y="116.84" size="1.27" layer="95" xref="yes"/>
+</segment>
+<segment>
+<pinref part="D9" gate="G$1" pin="A"/>
+<wire x1="116.84" y1="86.36" x2="114.3" y2="86.36" width="0.1524" layer="91"/>
+<label x="114.3" y="86.36" size="1.27" layer="95" rot="R180" xref="yes"/>
+</segment>
+</net>
+<net name="DIODO-6" class="0">
+<segment>
+<pinref part="IC3" gate="A" pin="QF"/>
+<wire x1="78.74" y1="114.3" x2="81.28" y2="114.3" width="0.1524" layer="91"/>
+<label x="81.28" y="114.3" size="1.27" layer="95" xref="yes"/>
+</segment>
+<segment>
+<pinref part="D10" gate="G$1" pin="A"/>
+<wire x1="116.84" y1="76.2" x2="114.3" y2="76.2" width="0.1524" layer="91"/>
+<label x="114.3" y="76.2" size="1.27" layer="95" rot="R180" xref="yes"/>
+</segment>
+</net>
+<net name="DIODO-7" class="0">
+<segment>
+<pinref part="IC3" gate="A" pin="QG"/>
+<wire x1="78.74" y1="111.76" x2="81.28" y2="111.76" width="0.1524" layer="91"/>
+<label x="81.28" y="111.76" size="1.27" layer="95" xref="yes"/>
+</segment>
+<segment>
+<pinref part="D11" gate="G$1" pin="A"/>
+<wire x1="116.84" y1="66.04" x2="114.3" y2="66.04" width="0.1524" layer="91"/>
+<label x="114.3" y="66.04" size="1.27" layer="95" rot="R180" xref="yes"/>
+</segment>
+</net>
+<net name="DIODO-8" class="0">
+<segment>
+<pinref part="IC3" gate="A" pin="QH"/>
+<wire x1="78.74" y1="109.22" x2="81.28" y2="109.22" width="0.1524" layer="91"/>
+<label x="81.28" y="109.22" size="1.27" layer="95" xref="yes"/>
+</segment>
+<segment>
+<pinref part="D12" gate="G$1" pin="A"/>
+<wire x1="116.84" y1="55.88" x2="114.3" y2="55.88" width="0.1524" layer="91"/>
+<label x="114.3" y="55.88" size="1.27" layer="95" rot="R180" xref="yes"/>
+</segment>
+</net>
+<net name="N$7" class="0">
+<segment>
+<pinref part="D5" gate="G$1" pin="C"/>
+<pinref part="R3" gate="G$1" pin="2"/>
+<wire x1="124.46" y1="127" x2="127" y2="127" width="0.1524" layer="91"/>
+</segment>
+</net>
+<net name="N$8" class="0">
+<segment>
+<pinref part="D6" gate="G$1" pin="C"/>
+<pinref part="R6" gate="G$1" pin="2"/>
+<wire x1="124.46" y1="116.84" x2="127" y2="116.84" width="0.1524" layer="91"/>
+</segment>
+</net>
+<net name="N$9" class="0">
+<segment>
+<pinref part="D7" gate="G$1" pin="C"/>
+<pinref part="R4" gate="G$1" pin="2"/>
+<wire x1="124.46" y1="106.68" x2="127" y2="106.68" width="0.1524" layer="91"/>
+</segment>
+</net>
+<net name="N$11" class="0">
+<segment>
+<pinref part="D8" gate="G$1" pin="C"/>
+<pinref part="R5" gate="G$1" pin="2"/>
+<wire x1="124.46" y1="96.52" x2="127" y2="96.52" width="0.1524" layer="91"/>
+</segment>
+</net>
+<net name="N$12" class="0">
+<segment>
+<pinref part="D9" gate="G$1" pin="C"/>
+<pinref part="R7" gate="G$1" pin="2"/>
+<wire x1="124.46" y1="86.36" x2="127" y2="86.36" width="0.1524" layer="91"/>
+</segment>
+</net>
+<net name="N$13" class="0">
+<segment>
+<pinref part="D10" gate="G$1" pin="C"/>
+<pinref part="R8" gate="G$1" pin="2"/>
+<wire x1="124.46" y1="76.2" x2="127" y2="76.2" width="0.1524" layer="91"/>
+</segment>
+</net>
+<net name="N$14" class="0">
+<segment>
+<pinref part="D11" gate="G$1" pin="C"/>
+<pinref part="R9" gate="G$1" pin="2"/>
+<wire x1="124.46" y1="66.04" x2="127" y2="66.04" width="0.1524" layer="91"/>
+</segment>
+</net>
+<net name="N$15" class="0">
+<segment>
+<pinref part="D12" gate="G$1" pin="C"/>
+<pinref part="R10" gate="G$1" pin="2"/>
+<wire x1="124.46" y1="55.88" x2="127" y2="55.88" width="0.1524" layer="91"/>
+</segment>
+</net>

Commit message: base
Connections:
- removed net N$5: IC3A.SER
- new net SR1: IC2A.QH*, IC3A.SER
- net GND: now also R10.1, R3.1, R4.1, R5.1, R6.1, R7.1, R8.1, R9.1, U$6.GND
Other:
- moved on the sheet: IC2P, IC3, IC3P
