File: hardware/electronics/Base/base.sch (EAGLE design)
At the start: 41 parts, among them IC1 7805T, IC2 74LS595D, IC3 74LS595D, IC4 74LS595D

Commit message: base+
Parts:
- added SV1, SV2, SV3, SV4: (no value), con-lstb:MA03-2
Connections:
- new net ALERT-1: SV1.5
- new net ALERT-2: SV3.5
- new net ALERT-3: SV2.5
- new net ALERT-4: SV4.5
- new net N$22: SV3.3
- new net N$25: SV1.3
- new net N$34: SV4.3
- new net N$37: SV2.3
- new net SCL: SV1.2, SV2.2, SV3.2, SV4.2
- new net SDA: SV1.4, SV2.4, SV3.4, SV4.4
- net 3.3V: now also SV1.6, SV2.6, SV3.6, SV4.6
- net GND: now also SV1.1, SV2.1, SV3.1, SV4.1
Other:
- note added: "Sensori di linea"
- moved on the sheet: X1-1, X1-2, X3-1, X3-2, X4-1, X4-2

Commit message: Base
Connections:
- net DIODO-1 renamed LED-1
- net DIODO-2 renamed LED-2
- net DIODO-3 renamed LED-3
- net DIODO-4 renamed LED-4
- net DIODO-5 renamed LED-5
- net DIODO-6 renamed LED-6
- net DIODO-7 renamed LED-7
- net DIODO-8 renamed LED-8
- removed net N$10: IC4A.SER
- new net SR2: IC3A.QH*, IC4A.SER
Other:
- note added: "Led segnalazione"
- note added: "Shift register"
- note added: "Shift register led"
- moved on the sheet: 5V, C1, C2, C3, C4, C5, D1, D10, D11, D12, D2, D3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

Commit message: Collegate le linee alla basa
Connections:
- removed net N$22: SV3.3
- removed net N$25: SV1.3
- removed net N$34: SV4.3
- removed net N$37: SV2.3
- net 3.3V: now also SV2.3, U$2.3.3V
- net GND: now also SV1.3
- net SCL: now also SV4.3, U$2.19/A5/T/SCL0
- net SDA: now also SV3.3, U$2.18/A4/T/SDA0
Changed lines of the file:
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@@
 <?xml version="1.0" encoding="utf-8"?>
 <!DOCTYPE eagle SYSTEM "eagle.dtd">
-<eagle version="8.6.3">
+<eagle version="8.6.0">
 <drawing>
 <settings>
@@
 <part name="SUPPLY16" library="SparkFun-PowerSymbols" deviceset="3.3V" device=""/>
 <part name="SUPPLY17" library="SparkFun-PowerSymbols" deviceset="3.3V" device=""/>
+<part name="SUPPLY18" library="SparkFun-PowerSymbols" deviceset="3.3V" device=""/>
 </parts>
 <sheets>
@@
 <wire x1="160.02" y1="58.42" x2="160.02" y2="88.9" width="1.27" layer="96" style="longdash"/>
 <wire x1="160.02" y1="58.42" x2="220.98" y2="58.42" width="1.27" layer="96" style="longdash"/>
-<text x="175.26" y="101.6" size="2.54" layer="99">Shift register motori</text>
+<text x="180.34" y="101.6" size="2.54" layer="99">Shift register motori</text>
 <wire x1="160.02" y1="88.9" x2="160.02" y2="106.68" width="1.27" layer="96" style="longdash"/>
 <wire x1="160.02" y1="106.68" x2="220.98" y2="106.68" width="1.27" layer="96" style="longdash"/>
@@
 <instance part="SUPPLY16" gate="G$1" x="213.36" y="149.86" rot="R90"/>
 <instance part="SUPPLY17" gate="G$1" x="213.36" y="132.08" rot="R90"/>
+<instance part="SUPPLY18" gate="G$1" x="246.38" y="147.32" rot="R270"/>
 </instances>
 <busses>
@@
 <label x="238.76" y="144.78" size="1.27" layer="95" xref="yes"/>
 </segment>
+<segment>
+<pinref part="SV1" gate="1" pin="3"/>
+<wire x1="195.58" y1="147.32" x2="198.12" y2="147.32" width="0.1524" layer="91"/>
+<label x="198.12" y="147.32" size="1.27" layer="95" xref="yes"/>
+</segment>
 </net>
 <net name="3.3V" class="0">
@@
 <pinref part="SUPPLY17" gate="G$1" pin="3.3V"/>
 </segment>
+<segment>
+<pinref part="SV2" gate="1" pin="3"/>
+<wire x1="236.22" y1="147.32" x2="246.38" y2="147.32" width="0.1524" layer="91"/>
+<pinref part="SUPPLY18" gate="G$1" pin="3.3V"/>
+</segment>
+<segment>
+<pinref part="U$2" gate="G$1" pin="3.3V"/>
+<pinref part="SUPPLY13" gate="G$1" pin="3.3V"/>
+<wire x1="142.24" y1="154.94" x2="144.78" y2="154.94" width="0.1524" layer="91"/>
+</segment>
 </net>
 <net name="N$2" class="0">
@@
 <label x="218.44" y="129.54" size="1.27" layer="95" rot="R180" xref="yes"/>
 </segment>
+<segment>
+<pinref part="SV3" gate="1" pin="3"/>
+<wire x1="195.58" y1="129.54" x2="198.12" y2="129.54" width="0.1524" layer="91"/>
+<label x="198.12" y="129.54" size="1.27" layer="95" xref="yes"/>
+</segment>
+<segment>
+<pinref part="U$2" gate="G$1" pin="18/A4/T/SDA0"/>
+<junction x="96.52" y="111.76"/>
+<label x="96.52" y="111.76" size="1.27" layer="95" rot="R180" xref="yes"/>
+</segment>
 </net>
 <net name="SCL" class="0">
@@
 <label x="218.44" y="144.78" size="1.27" layer="95" rot="R180" xref="yes"/>
 </segment>
-</net>
-<net name="N$22" class="0">
-<segment>
-<pinref part="SV3" gate="1" pin="3"/>
-<wire x1="195.58" y1="129.54" x2="198.12" y2="129.54" width="0.1524" layer="91"/>
-<label x="198.12" y="129.54" size="1.27" layer="95" xref="yes"/>
+<segment>
+<pinref part="SV4" gate="1" pin="3"/>
+<wire x1="236.22" y1="129.54" x2="238.76" y2="129.54" width="0.1524" layer="91"/>
+<label x="238.76" y="129.54" size="1.27" layer="95" xref="yes"/>
+</segment>
+<segment>
+<pinref part="U$2" gate="G$1" pin="19/A5/T/SCL0"/>
+<junction x="96.52" y="109.22"/>
+<label x="96.52" y="109.22" size="1.27" layer="95" rot="R180" xref="yes"/>
 </segment>
 </net>
@@
 </segment>
 </net>
-<net name="N$25" class="0">
-<segment>
-<pinref part="SV1" gate="1" pin="3"/>
-<wire x1="195.58" y1="147.32" x2="198.12" y2="147.32" width="0.1524" layer="91"/>
-<label x="198.12" y="147.32" size="1.27" layer="95" xref="yes"/>
-</segment>
-</net>
 <net name="ALERT-1" class="0">
 <segment>
@@
 </segment>
 </net>
-<net name="N$34" class="0">
-<segment>
-<pinref part="SV4" gate="1" pin="3"/>
-<wire x1="236.22" y1="129.54" x2="238.76" y2="129.54" width="0.1524" layer="91"/>
-<label x="238.76" y="129.54" size="1.27" layer="95" xref="yes"/>
-</segment>
-</net>
 <net name="ALERT-4" class="0">
 <segment>
@@
 </segment>
 </net>
-<net name="N$37" class="0">
-<segment>
-<pinref part="SV2" gate="1" pin="3"/>
-<wire x1="236.22" y1="147.32" x2="238.76" y2="147.32" width="0.1524" layer="91"/>
-<label x="238.76" y="147.32" size="1.27" layer="95" xref="yes"/>
-</segment>
-</net>
